File: KiCad/triple_cp2108/2108.sch (KiCad schematic (older format))
At the start: 1 part

Commit message: Parts importing in prgs.
Parts:
- added J? (x4): RJ12, symbol Connector:RJ12
- gave numbers to parts that had none: 1
Connections:
- net VBUS_5V: now reaches IC1.61 (VBUS)
- net D+: now reaches IC1.62 (D+)
- net D-: now reaches IC1.63 (D-)
- new net P1_1: J?.1
- new net P1_2: J?.2
- new net P1_3: J?.3
- new net P1_4: J?.4
- new net P1_5: J?.5
- new net P1_6: J?.6
- new net P2_1: J?.1
- new net P2_2: J?.2
- new net P2_3: J?.3
- new net P2_4: J?.4
- new net P2_5: J?.5
- new net P2_6: J?.6
- new net P3_1: J?.1
- new net P3_2: J?.2
- new net P3_3: J?.3
- new net P3_4: J?.4
- new net P3_5: J?.5
- new net P3_6: J?.6
- new net P4_1: J?.1
- new net P4_2: J?.2
- new net P4_3: J?.3
- new net P4_4: J?.4
- new net P4_5: J?.5
- new net P4_6: J?.6
Other:
- moved on the sheet: IC1
Changed lines of the file:
@@
 $Descr A4 11693 8268
 encoding utf-8
-Sheet 3 3
+Sheet 2 3
 Title ""
 Date ""
@@
 $EndDescr
 $Comp
-L Samacsys:CP2108-B03-GMR IC?
+L Samacsys:CP2108-B03-GMR IC1
 U 1 1 5FEF563A
-P 4700 2750
-AR Path="/5FEF445C/5FEF563A" Ref="IC?"  Part="1"
-AR Path="/5FEFA5BE/5FEF563A" Ref="IC?"  Part="1"
-F 0 "IC?" H 6944 1996 50  0000 L CNN
-F 1 "CP2108-B03-GMR" H 6944 1905 50  0000 L CNN
-F 2 "QFN50P900X900X90-65N-D" H 6750 3250 50  0001 L CNN
-F 3 "https://www.silabs.com/documents/public/data-sheets/cp2108-datasheet.pdf" H 6750 3150 50  0001 L CNN
-F 4 "SILICON LABS - CP2108-B03-GMR - Interface Bridges, USB to UART, 3 V, 3.6 V, QFN-EP, 64 Pins, -40 C" H 6750 3050 50  0001 L CNN "Description"
-F 5 "0.9" H 6750 2950 50  0001 L CNN "Height"
-F 6 "634-CP2108-B03-GMR" H 6750 2850 50  0001 L CNN "Mouser Part Number"
-F 7 "https://www.mouser.co.uk/ProductDetail/Silicon-Labs/CP2108-B03-GMR?qs=wd5RIQLrsJhyaTycraVyrA%3D%3D" H 6750 2750 50  0001 L CNN "Mouser Price/Stock"
-F 8 "Silicon Labs" H 6750 2650 50  0001 L CNN "Manufacturer_Name"
-F 9 "CP2108-B03-GMR" H 6750 2550 50  0001 L CNN "Manufacturer_Part_Number"
-	1    4700 2750
+P 1900 2500
+AR Path="/5FEF445C/5FEF563A" Ref="IC1"  Part="1"
+AR Path="/5FEFA5BE/5FEF563A" Ref="IC2"  Part="1"
+F 0 "IC1" H 4144 1746 50  0000 L CNN
+F 1 "CP2108-B03-GMR" H 4144 1655 50  0000 L CNN
+F 2 "QFN50P900X900X90-65N-D" H 3950 3000 50  0001 L CNN
+F 3 "https://www.silabs.com/documents/public/data-sheets/cp2108-datasheet.pdf" H 3950 2900 50  0001 L CNN
+F 4 "SILICON LABS - CP2108-B03-GMR - Interface Bridges, USB to UART, 3 V, 3.6 V, QFN-EP, 64 Pins, -40 C" H 3950 2800 50  0001 L CNN "Description"
+F 5 "0.9" H 3950 2700 50  0001 L CNN "Height"
+F 6 "634-CP2108-B03-GMR" H 3950 2600 50  0001 L CNN "Mouser Part Number"
+F 7 "https://www.mouser.co.uk/ProductDetail/Silicon-Labs/CP2108-B03-GMR?qs=wd5RIQLrsJhyaTycraVyrA%3D%3D" H 3950 2500 50  0001 L CNN "Mouser Price/Stock"
+F 8 "Silicon Labs" H 3950 2400 50  0001 L CNN "Manufacturer_Name"
+F 9 "CP2108-B03-GMR" H 3950 2300 50  0001 L CNN "Manufacturer_Part_Number"
+	1    1900 2500
 	1    0    0    -1
 $EndComp
+Wire Wire Line
+	2400 1800 2400 1650
+Wire Wire Line
+	2500 1800 2500 1650
+Text Label 2400 1650 1    50   ~ 0
+D-
+Text Label 2500 1650 1    50   ~ 0
+D+
+Wire Wire Line
+	2600 1800 2600 1650
+Text Label 2600 1650 1    50   ~ 0
+VBUS_5V
+$Comp
+L Connector:RJ12 J?
+U 1 1 5FE61D47
+P 10600 1100
+F 0 "J?" H 10657 1667 50  0000 C CNN
+F 1 "RJ12" H 10657 1576 50  0000 C CNN
+F 2 "" V 10600 1125 50  0001 C CNN
+F 3 "~" V 10600 1125 50  0001 C CNN
+	1    10600 1100
+	-1   0    0    1
+$EndComp
+Wire Wire Line
+	10200 1400 10050 1400
+Text Label 10050 1400 2    50   ~ 0
+P1_6
+Wire Wire Line
+	10200 1300 10050 1300
+Text Label 10050 1300 2    50   ~ 0
+P1_5
+Wire Wire Line
+	10200 1200 10050 1200
+Text Label 10050 1200 2    50   ~ 0
+P1_4
+Wire Wire Line
+	10200 1100 10050 1100
+Text Label 10050 1100 2    50   ~ 0
+P1_3
+Wire Wire Line
+	10200 1000 10050 1000
+Text Label 10050 1000 2    50   ~ 0
+P1_2
+Wire Wire Line
+	10200 900  10050 900
+Text Label 10050 900  2    50   ~ 0
+P1_1
+$Comp
+L Connector:RJ12 J?
+U 1 1 5FE641F2
+P 10600 2150
+F 0 "J?" H 10657 2717 50  0000 C CNN
+F 1 "RJ12" H 10657 2626 50  0000 C CNN
+F 2 "" V 10600 2175 50  0001 C CNN
+F 3 "~" V 10600 2175 50  0001 C CNN
+	1    10600 2150
+	-1   0    0    1
+$EndComp
+Wire Wire Line
+	10200 2450 10050 2450
+Text Label 10050 2450 2    50   ~ 0
+P2_6
+Wire Wire Line
+	10200 2350 10050 2350
+Text Label 10050 2350 2    50   ~ 0
+P2_5
+Wire Wire Line
+	10200 2250 10050 2250
+Text Label 10050 2250 2    50   ~ 0
+P2_4
+Wire Wire Line
+	10200 2150 10050 2150
+Text Label 10050 2150 2    50   ~ 0
+P2_3
+Wire Wire Line
+	10200 2050 10050 2050
+Text Label 10050 2050 2    50   ~ 0
+P2_2
+Wire Wire Line
+	10200 1950 10050 1950
+Text Label 10050 1950 2    50   ~ 0
+P2_1
+$Comp
+L Connector:RJ12 J?
+U 1 1 5FE68DE0
+P 10600 3200
+F 0 "J?" H 10657 3767 50  0000 C CNN
+F 1 "RJ12" H 10657 3676 50  0000 C CNN
+F 2 "" V 10600 3225 50  0001 C CNN
+F 3 "~" V 10600 3225 50  0001 C CNN
+	1    10600 3200
+	-1   0    0    1
+$EndComp
+Wire Wire Line
+	10200 3500 10050 3500
+Text Label 10050 3500 2    50   ~ 0
+P3_6
+Wire Wire Line
+	10200 3400 10050 3400
+Text Label 10050 3400 2    50   ~ 0
+P3_5
+Wire Wire Line
+	10200 3300 10050 3300
+Text Label 10050 3300 2    50   ~ 0
+P3_4
+Wire Wire Line
+	10200 3200 10050 3200
+Text Label 10050 3200 2    50   ~ 0
+P3_3
+Wire Wire Line
+	10200 3100 10050 3100
+Text Label 10050 3100 2    50   ~ 0
+P3_2
+Wire Wire Line
+	10200 3000 10050 3000
+Text Label 10050 3000 2    50   ~ 0
+P3_1
+$Comp
+L Connector:RJ12 J?
+U 1 1 5FE68DF2
+P 10600 4250
+F 0 "J?" H 10657 4817 50  0000 C CNN
+F 1 "RJ12" H 10657 4726 50  0000 C CNN
+F 2 "" V 10600 4275 50  0001 C CNN
+F 3 "~" V 10600 4275 50  0001 C CNN
+	1    10600 4250
+	-1   0    0    1
+$EndComp
+Wire Wire Line
+	10200 4550 10050 4550
+Text Label 10050 4550 2    50   ~ 0
+P4_6
+Wire Wire Line
+	10200 4450 10050 4450
+Text Label 10050 4450 2    50   ~ 0
+P4_5
+Wire Wire Line
+	10200 4350 10050 4350
+Text Label 10050 4350 2    50   ~ 0
+P4_4
+Wire Wire Line
+	10200 4250 10050 4250
+Text Label 10050 4250 2    50   ~ 0
+P4_3
+Wire Wire Line
+	10200 4150 10050 4150
+Text Label 10050 4150 2    50   ~ 0
+P4_2
+Wire Wire Line
+	10200 4050 10050 4050
+Text Label 10050 4050 2    50   ~ 0
+P4_1
 $EndSCHEMATC

Commit message: 2108 in prgs.
Parts:
- added C? (x5): 0.1u, symbol Device:C
- added U?: SP3243, Package_SO:SSOP-28_5.3x10.2mm_P0.65mm, symbol triple_cp2108_specific:SP3243
Connections:
- net P1_1: no longer J?.1
- net P1_2: no longer J?.2
- net P1_3: no longer J?.3
- net P1_4: no longer J?.4
- net P1_5: no longer J?.5
- net P1_6: no longer J?.6
- net P2_1: no longer J?.1
- net P2_2: no longer J?.2
- net P2_3: no longer J?.3
- net P2_4: no longer J?.4
- net P2_5: no longer J?.5
- net P2_6: no longer J?.6
- net P3_1: no longer J?.1
- net P3_2: no longer J?.2
- net P3_3: no longer J?.3
- net P3_4: no longer J?.4
- net P3_5: no longer J?.5
- net P3_6: no longer J?.6
- net P4_1: no longer J?.1
- net P4_2: no longer J?.2
- net P4_3: no longer J?.3
- net P4_4: no longer J?.4
- net P4_5: no longer J?.5
- net P4_6: no longer J?.6
- new net: C?.2, U?.1 (C2+)
- new net: C?.1, U?.2 (C2-)
- new net: C?.1, U?.24 (C1-)
- new net: C?.1, U?.27 (V+)
- new net: C?.2, U?.28 (C1+)
- new net: C?.1, U?.3 (V-)
- new net 3V3_NET: C?.2, U?.23 (~ONLINE), U?.26 (VCC)
- new net GND: C?.1, C?.2, C?.2, U?.25 (GND)
- no-connect marks 0 -> 1
Other:
- moved on the sheet: IC1, J?

Commit message: 2108 in prgs.
Parts:
- removed J? (x3): RJ12, symbol Connector:RJ12
- added C? (x15): 0.1u, symbol Device:C
- added J? (x4): Screw_Terminal_01x09, symbol Connector:Screw_Terminal_01x09
- added J? (x3): RJ12, symbol Connector:RJ12
- added R? (x8): 0, symbol Device:R
- added R? (x8): NC, symbol Device:R
- added U? (x3): SP3243, Package_SO:SSOP-28_5.3x10.2mm_P0.65mm, symbol triple_cp2108_specific:SP3243
Connections:
- net 3V3_NET: now also C?.2, C?.2, C?.2, U?.23 (~ONLINE), U?.23 (~ONLINE), U?.23 (~ONLINE), U?.26 (VCC), U?.26 (VCC), U?.26 (VCC)
- net GND: now also IC1.2 (VSSHD), IC1.25 (VSS_1), IC1.59 (VSS_2), IC1.65 (VSS_3), J?.3, J?.4, C?.1, C?.1, C?.1, C?.2, C?.2, C?.2, C?.2, C?.2, C?.2, J?.1 (Pin_1), J?.1 (Pin_1), J?.1 (Pin_1), J?.1 (Pin_1), J?.3, J?.3, J?.3, J?.4, J?.4, J?.4, U?.25 (GND), U?.25 (GND), U?.25 (GND)
- net VBUS_5V: now also IC1.60 (VREGIN)
- net at J?.2: now also R?.2, R?.2
- net at J?.5: now also R?.2, R?.2
- net RTS232_1: now reaches U?.10 (T2OUT)
- net RTS232_1: now also J?.4 (Pin_4), U?.10 (T2OUT), U?.10 (T2OUT), U?.10 (T2OUT)
- net DTR232_1: now reaches U?.11 (T3OUT)
- net DTR232_1: now also J?.6 (Pin_6), U?.11 (T3OUT), U?.11 (T3OUT), U?.11 (T3OUT)
- net DTR1: now reaches U?.12 (T3IN)
- net DTR1: now also IC1.53 (DTR0), U?.12 (T3IN), U?.12 (T3IN), U?.12 (T3IN)
- net RTS1: now reaches U?.13 (T2IN)
- net RTS1: now also IC1.55 (RTS0), U?.13 (T2IN), U?.13 (T2IN), U?.13 (T2IN)
- net TXD1: now reaches U?.14 (T1IN)
- net TXD1: now also IC1.57 (TX0), U?.14 (T1IN), U?.14 (T1IN), U?.14 (T1IN)
- net RI1: now reaches U?.15 (R5OUT)
- net RI1: now also IC1.50 (RI0), U?.15 (R5OUT), U?.15 (R5OUT), U?.15 (R5OUT)
- net DCD1: now reaches U?.16 (R4OUT)
- net DCD1: now also IC1.51 (DCD0), U?.16 (R4OUT), U?.16 (R4OUT), U?.16 (R4OUT)
- net DSR1: now reaches U?.17 (R3OUT)
- net DSR1: now also IC1.52 (DSR0), U?.17 (R3OUT), U?.17 (R3OUT), U?.17 (R3OUT)
- net CTS1: now reaches U?.18 (R2OUT)
- net CTS1: now also IC1.54 (CTS0), U?.18 (R2OUT), U?.18 (R2OUT), U?.18 (R2OUT)
- net RXD1: now reaches U?.19 (R1OUT)
- net RXD1: now also IC1.56 (RX0), U?.19 (R1OUT), U?.19 (R1OUT), U?.19 (R1OUT)
- net ~SUSPEND: now reaches U?.22 (~SHUTDOWN)
- net ~SUSPEND: now also IC1.19 (~SUSPEND), U?.22 (~SHUTDOWN), U?.22 (~SHUTDOWN), U?.22 (~SHUTDOWN)
- net RXD232_1: now reaches U?.4 (R1IN)
- net RXD232_1: now also J?.3 (Pin_3), R?.1, R?.1, U?.4 (R1IN), U?.4 (R1IN), U?.4 (R1IN)
- net CTS232_1: now reaches U?.5 (R2IN)
- net CTS232_1: now also J?.5 (Pin_5), U?.5 (R2IN), U?.5 (R2IN), U?.5 (R2IN)
- net DSR232_1: now reaches U?.6 (R3IN)
- net DSR232_1: now also J?.7 (Pin_7), U?.6 (R3IN), U?.6 (R3IN), U?.6 (R3IN)
- net DCD232_1: now reaches U?.7 (R4IN)
- net DCD232_1: now also J?.8 (Pin_8), U?.7 (R4IN), U?.7 (R4IN), U?.7 (R4IN)
- net RI232_1: now reaches U?.8 (R5IN)
- net RI232_1: now also J?.9 (Pin_9), U?.8 (R5IN), U?.8 (R5IN), U?.8 (R5IN)
- net TXD232_1: now reaches U?.9 (T1OUT)
- net TXD232_1: now also J?.2 (Pin_2), R?.1, R?.1, U?.9 (T1OUT), U?.9 (T1OUT), U?.9 (T1OUT)
- net RXD4: now reaches IC1.1 (RX3)
- net DTR4: now reaches IC1.10 (DTR3)
- net RI3: now reaches IC1.11 (RI2)
- net DCD3: now reaches IC1.12 (DCD2)
- net CTS3: now reaches IC1.13 (CTS2)
- net RTS3: now reaches IC1.14 (RTS2)
- net RXD3: now reaches IC1.15 (RX2)
- net TXD3: now reaches IC1.16 (TX2)
- net DSR3: now reaches IC1.17 (DSR2)
- net DTR3: now reaches IC1.18 (DTR2)
- net VIO: now reaches IC1.24 (VIO_1)
- net VIO: now also IC1.3 (VIOHD), IC1.39 (VIO_2)
- net TXD4: now reaches IC1.4 (TX3)
- net RI2: now reaches IC1.42 (RI1)
- net DCD2: now reaches IC1.43 (DCD1)
- net DSR2: now reaches IC1.44 (DSR1)
- net DTR2: now reaches IC1.45 (DTR1)
- net CTS2: now reaches IC1.46 (CTS1)
- net RTS2: now reaches IC1.47 (RTS1)
- net RXD2: now reaches IC1.48 (RX1)
- net TXD2: now reaches IC1.49 (TX1)
- net CTS4: now reaches IC1.5 (CTS3)
- net RTS4: now reaches IC1.6 (RTS3)
- net ~RESET: now reaches IC1.64 (~RESET)
- net RI4: now reaches IC1.7 (RI3)
- net DCD4: now reaches IC1.8 (DCD3)
- net DSR4: now reaches IC1.9 (DSR3)
- new net: J?.2, R?.2, R?.2 (x3)
- new net: J?.5, R?.2, R?.2 (x3)
- new net: C?.1, U?.2 (C2-) (x3)
- new net: C?.2, U?.1 (C2+) (x3)
- new net: C?.1, U?.24 (C1-) (x3)
- new net: C?.2, U?.28 (C1+) (x3)
- new net: C?.1, U?.27 (V+) (x3)
- new net: C?.1, U?.3 (V-) (x3)
- new net CTS232_2: J?.5 (Pin_5)
- new net CTS232_3: J?.5 (Pin_5)
- new net CTS232_4: J?.5 (Pin_5)
- new net DCD232_2: J?.8 (Pin_8)
- new net DCD232_3: J?.8 (Pin_8)
- new net DCD232_4: J?.8 (Pin_8)
- new net DSR232_2: J?.7 (Pin_7)
- new net DSR232_3: J?.7 (Pin_7)
- new net DSR232_4: J?.7 (Pin_7)
- new net DTR232_2: J?.6 (Pin_6)
- new net DTR232_3: J?.6 (Pin_6)
- new net DTR232_4: J?.6 (Pin_6)
- new net RI232_2: J?.9 (Pin_9)
- new net RI232_3: J?.9 (Pin_9)
- new net RI232_4: J?.9 (Pin_9)
- new net RTS232_2: J?.4 (Pin_4)
- new net RTS232_3: J?.4 (Pin_4)
- new net RTS232_4: J?.4 (Pin_4)
- new net RXD232_2: J?.3 (Pin_3), R?.1, R?.1
- new net RXD232_3: J?.3 (Pin_3), R?.1, R?.1
- new net RXD232_4: J?.3 (Pin_3), R?.1, R?.1
- new net TXD232_2: J?.2 (Pin_2), R?.1, R?.1
- new net TXD232_3: J?.2 (Pin_2), R?.1, R?.1
- new net TXD232_4: J?.2 (Pin_2), R?.1, R?.1
- no-connect marks 1 -> 18
Other:
- moved on the sheet: C?, IC1, J?, U?

Commit message: 2108 done
Parts:
- added C? (x6): 0.1u, symbol Device:C
- added C? (x3): 4.7u, symbol Device:C
- added D? (x4): RED, symbol Device:LED
- added D? (x4): GREEN, symbol Device:LED
- added R? (x8): R, symbol Device:R
- added R?: 1K, symbol Device:R
Connections:
- net VIO is gone; now on net 3V3_NET: IC1.24 (VIO_1), IC1.3 (VIOHD), IC1.39 (VIO_2)
- net 3V3_NET: now also IC1.58 (VDD), C?.2, C?.2, C?.2, C?.2, C?.2, C?.2, C?.2, R?.1, R?.1, R?.1, R?.1, R?.1, R?.1, R?.1, R?.1, R?.1
- net GND: now also C?.1, C?.1, C?.1, C?.1, C?.1, C?.1, C?.1, C?.1, C?.1
- net VBUS_5V: now also C?.2, C?.2
- net ~RESET: now also R?.2
- net GPIO15: now reaches IC1.21 (GPIO.15)
- net GPIO14: now reaches IC1.22 (GPIO.14)
- net RXD3_LED: now reaches IC1.23 (GPIO.13)
- net RXD3_LED: now also IC1.29 (GPIO.9), D?.1 (K)
- net TXD3_LED: now reaches IC1.26 (GPIO.12)
- net TXD3_LED: now also IC1.30 (GPIO.8), D?.1 (K)
- net GPIO11: now reaches IC1.27 (GPIO.11)
- net GPIO10: now reaches IC1.28 (GPIO.10)
- net GPIO7: now reaches IC1.31 (GPIO.7)
- net GPIO6: now reaches IC1.32 (GPIO.6)
- net RXD2_LED: now reaches IC1.33 (GPIO.5)
- net RXD2_LED: now also D?.1 (K)
- net TXD2_LED: now reaches IC1.34 (GPIO.4)
- net TXD2_LED: now also D?.1 (K)
- net GPIO3: now reaches IC1.37 (GPIO.3)
- net GPIO2: now reaches IC1.38 (GPIO.2)
- net RXD1_LED: now reaches IC1.40 (GPIO.1)
- net RXD1_LED: now also D?.1 (K)
- net TXD1_LED: now reaches IC1.41 (GPIO.0)
- net TXD1_LED: now also D?.1 (K)
- new net: D?.2 (A), R?.2 (x8)
- new net RXD4_LED: D?.1 (K)
- new net TXD4_LED: D?.1 (K)
- no-connect marks 18 -> 19
Other:
- moved on the sheet: IC1

Commit message: GPIO Consolidation in prgs.
Changed lines of the file:
@@
 encoding utf-8
 Sheet 2 4
-Title ""
-Date ""
-Rev ""
+Title "CP2108 Evaluation board"
+Date "2020-12-26"
+Rev "0"
 Comp ""
 Comment1 ""
@@
 Text Label 1850 1750 1    50   ~ 0
 VDD
-Text Label 4850 2100 2    50   ~ 0
-VDD
-Wire Wire Line
-	4850 2100 4950 2100
-Text Label 5050 2100 0    50   ~ 0
-3V3_NET
-Wire Wire Line
-	4950 2100 4950 2200
-Wire Wire Line
-	4950 2200 5050 2200
-Connection ~ 4950 2100
-Wire Wire Line
-	4950 2100 5050 2100
-Text Label 5050 2200 0    50   ~ 0
-VIO
 $Comp
 L Device:C C?
@@
 Wire Wire Line
 	4950 4500 5400 4500
+Text HLabel 1100 650  0    50   Input ~ 0
+VBUS_5V
+Text Label 1300 650  0    50   ~ 0
+VBUS_5V
+Wire Wire Line
+	1300 650  1100 650
+Text HLabel 1100 750  0    50   Input ~ 0
+D-
+Text HLabel 1100 850  0    50   Input ~ 0
+D+
+Text Label 1300 750  0    50   ~ 0
+D-
+Text Label 1300 850  0    50   ~ 0
+D+
+Wire Wire Line
+	1100 750  1300 750
+Wire Wire Line
+	1100 850  1300 850
+Text HLabel 1100 950  0    50   Input ~ 0
+GND
+Wire Wire Line
+	1100 950  1300 950
+Wire Wire Line
+	1300 950  1300 1000
+$Comp
+L power:GND #PWR?
+U 1 1 609A9296
+P 1300 1000
+AR Path="/5FEF445C/609A9296" Ref="#PWR?"  Part="1"
+AR Path="/5FEFA5BE/609A9296" Ref="#PWR?"  Part="1"
+AR Path="/6001CD0C/609A9296" Ref="#PWR?"  Part="1"
+F 0 "#PWR?" H 1300 750 50  0001 C CNN
+F 1 "GND" H 1305 827 50  0000 C CNN
+F 2 "" H 1300 1000 50  0001 C CNN
+F 3 "" H 1300 1000 50  0001 C CNN
+	1    1300 1000
+	1    0    0    -1
+$EndComp
+Wire Wire Line
+	4850 2100 4950 2100
+Text Label 5050 2100 0    50   ~ 0
+3V3_NET
+Wire Wire Line
+	4950 2100 4950 2200
+Wire Wire Line
+	4950 2200 5050 2200
+Connection ~ 4950 2100
+Wire Wire Line
+	4950 2100 5050 2100
+Text Label 5050 2200 0    50   ~ 0
+VIO
+Text Label 4850 2100 2    50   ~ 0
+VDD
+Text HLabel 2100 650  0    50   Input ~ 0
+GPIO2
+Text HLabel 2100 750  0    50   Input ~ 0
+GPIO3
+Text HLabel 2100 850  0    50   Input ~ 0
+GPIO6
+Text HLabel 2100 950  0    50   Input ~ 0
+GPIO7
+Text HLabel 2100 1050 0    50   Input ~ 0
+GPIO10
+Text HLabel 2100 1150 0    50   Input ~ 0
+GPIO11
+Text HLabel 2100 1250 0    50   Input ~ 0
+GPIO14
+Text HLabel 2100 1350 0    50   Input ~ 0
+GPIO15
+Text Label 2300 650  0    50   ~ 0
+GPIO2
+Wire Wire Line
+	2300 650  2100 650
+Text Label 2300 750  0    50   ~ 0
+GPIO3
+Text Label 2300 850  0    50   ~ 0
+GPIO6
+Wire Wire Line
+	2100 750  2300 750
+Wire Wire Line
+	2100 850  2300 850
+Text Label 2300 950  0    50   ~ 0
+GPIO7
+Wire Wire Line
+	2300 950  2100 950
+Text Label 2300 1050 0    50   ~ 0
+GPIO10
+Text Label 2300 1150 0    50   ~ 0
+GPIO11
+Wire Wire Line
+	2100 1050 2300 1050
+Wire Wire Line
+	2100 1150 2300 1150
+Text Label 2300 1250 0    50   ~ 0
+GPIO14
+Text Label 2300 1350 0    50   ~ 0
+GPIO15
+Wire Wire Line
+	2100 1250 2300 1250
+Wire Wire Line
+	2100 1350 2300 1350
 $EndSCHEMATC

Commit message: misc.
Parts:
- gave numbers to parts that had none: 74
Connections:
- net CTS1: no longer U12.18 (R2OUT), U13.18 (R2OUT), U14.18 (R2OUT)
- net CTS2: now also U12.18 (R2OUT)
- net CTS232_1: no longer U12.5 (R2IN), U13.5 (R2IN), U14.5 (R2IN)
- net CTS232_2: now also U12.5 (R2IN)
- net CTS232_3: now also U13.5 (R2IN)
- net CTS232_4: now also U14.5 (R2IN)
- net CTS3: now also U13.18 (R2OUT)
- net CTS4: now also U14.18 (R2OUT)
- net DCD1: no longer U12.16 (R4OUT), U13.16 (R4OUT), U14.16 (R4OUT)
- net DCD2: now also U12.16 (R4OUT)
- net DCD232_1: no longer U12.7 (R4IN), U13.7 (R4IN), U14.7 (R4IN)
- net DCD232_2: now also U12.7 (R4IN)
- net DCD232_3: now also U13.7 (R4IN)
- net DCD232_4: now also U14.7 (R4IN)
- net DCD3: now also U13.16 (R4OUT)
- net DCD4: now also U14.16 (R4OUT)
- net DSR1: no longer U12.17 (R3OUT), U13.17 (R3OUT), U14.17 (R3OUT)
- net DSR2: now also U12.17 (R3OUT)
- net DSR232_1: no longer U12.6 (R3IN), U13.6 (R3IN), U14.6 (R3IN)
- net DSR232_2: now also U12.6 (R3IN)
- net DSR232_3: now also U13.6 (R3IN)
- net DSR232_4: now also U14.6 (R3IN)
- net DSR3: now also U13.17 (R3OUT)
- net DSR4: now also U14.17 (R3OUT)
- net DTR1: no longer U12.12 (T3IN), U13.12 (T3IN), U14.12 (T3IN)
- net DTR2: now also U12.12 (T3IN)
- net DTR232_1: no longer U12.11 (T3OUT), U13.11 (T3OUT), U14.11 (T3OUT)
- net DTR232_2: now also U12.11 (T3OUT)
- net DTR232_3: now also U13.11 (T3OUT)
- net DTR232_4: now also U14.11 (T3OUT)
- net DTR3: now also U13.12 (T3IN)
- net DTR4: now also U14.12 (T3IN)
- net RI1: no longer U12.15 (R5OUT), U13.15 (R5OUT), U14.15 (R5OUT)
- net RI2: now also U12.15 (R5OUT)
- net RI232_1: no longer U12.8 (R5IN), U13.8 (R5IN), U14.8 (R5IN)
- net RI232_2: now also U12.8 (R5IN)
- net RI232_3: now also U13.8 (R5IN)
- net RI232_4: now also U14.8 (R5IN)
- net RI3: now also U13.15 (R5OUT)
- net RI4: now also U14.15 (R5OUT)
- net RTS1: no longer U12.13 (T2IN), U13.13 (T2IN), U14.13 (T2IN)
- net RTS2: now also U12.13 (T2IN)
- net RTS232_1: no longer U12.10 (T2OUT), U13.10 (T2OUT), U14.10 (T2OUT)
- net RTS232_2: now also U12.10 (T2OUT)
- net RTS232_3: now also U13.10 (T2OUT)
- net RTS232_4: now also U14.10 (T2OUT)
- net RTS3: now also U13.13 (T2IN)
- net RTS4: now also U14.13 (T2IN)
- net RXD1: no longer U12.19 (R1OUT), U13.19 (R1OUT), U14.19 (R1OUT)
- net RXD2: now also U12.19 (R1OUT)
- net RXD232_1: no longer U12.4 (R1IN), U13.4 (R1IN), U14.4 (R1IN)
- net RXD232_2: now also U12.4 (R1IN)
- net RXD232_3: now also U13.4 (R1IN)
- net RXD232_4: now also U14.4 (R1IN)
- net RXD3: now also U13.19 (R1OUT)
- net RXD4: now also U14.19 (R1OUT)
- net TXD1: no longer U12.14 (T1IN), U13.14 (T1IN), U14.14 (T1IN)
- net TXD2: now also U12.14 (T1IN)
- net TXD232_1: no longer U12.9 (T1OUT), U13.9 (T1OUT), U14.9 (T1OUT)
- net TXD232_2: now also U12.9 (T1OUT)
- net TXD232_3: now also U13.9 (T1OUT)
- net TXD232_4: now also U14.9 (T1OUT)
- net TXD3: now also U13.14 (T1IN)
- net TXD4: now also U14.14 (T1IN)
