File: KiCad/triple_cp2108/triple_cp2108.kicad_pcb (KiCad board)
At the start: 2 copper layers, 6 parts, among them IC1 CP2108-B03-GMR, IC2 CP2108-B03-GMR, U1 MIC5504-3.3YM5, U2 USB2514B_Bi

Commit message: Netlist generated
Parts:
- added C1: 18p, Capacitor_SMD:C_0805_2012Metric_Pad1.18x1.45mm_HandSolder, F.Cu at (54.9, -16.1)
- added C10: 0.1u, Capacitor_SMD:C_0805_2012Metric_Pad1.18x1.45mm_HandSolder, F.Cu at (-170.3, -180.0)
- added C11: 4.7u, Capacitor_SMD:C_0805_2012Metric_Pad1.18x1.45mm_HandSolder, F.Cu at (-177.2, -174.0)
- added C12: 0.1u, Capacitor_SMD:C_0805_2012Metric_Pad1.18x1.45mm_HandSolder, F.Cu at (-190.9, -159.9)
- added C13: 0.1u, Capacitor_SMD:C_0805_2012Metric_Pad1.18x1.45mm_HandSolder, F.Cu at (-212.8, -140.4)
- added C14: 0.1u, Capacitor_SMD:C_0805_2012Metric_Pad1.18x1.45mm_HandSolder, F.Cu at (-207.1, -146.4)
- added C15: 0.1u, Capacitor_SMD:C_0805_2012Metric_Pad1.18x1.45mm_HandSolder, F.Cu at (-175.1, -177.0)
- added C16: 4.7u, Capacitor_SMD:C_0805_2012Metric_Pad1.18x1.45mm_HandSolder, F.Cu at (-182.0, -174.0)
- added C17: 0.1u, Capacitor_SMD:C_0805_2012Metric_Pad1.18x1.45mm_HandSolder, F.Cu at (-212.8, -137.4)
- added C18: 0.1u, Capacitor_SMD:C_0805_2012Metric_Pad1.18x1.45mm_HandSolder, F.Cu at (-177.2, -171.0)
- added C19: 0.1u, Capacitor_SMD:C_0805_2012Metric_Pad1.18x1.45mm_HandSolder, F.Cu at (-240.0, -167.4)
- added C2: 18p, Capacitor_SMD:C_0805_2012Metric_Pad1.18x1.45mm_HandSolder, F.Cu at (50.1, -13.1)
- added C20: 0.1u, Capacitor_SMD:C_0805_2012Metric_Pad1.18x1.45mm_HandSolder, F.Cu at (-259.1, -168.7)
- added C21: 0.1u, Capacitor_SMD:C_0805_2012Metric_Pad1.18x1.45mm_HandSolder, F.Cu at (-191.6, -172.0)
- added C22: 0.1u, Capacitor_SMD:C_0805_2012Metric_Pad1.18x1.45mm_HandSolder, F.Cu at (-191.6, -169.0)
- added C23: 0.1u, Capacitor_SMD:C_0805_2012Metric_Pad1.18x1.45mm_HandSolder, F.Cu at (-254.0, -189.0)
- added C24: 0.1u, Capacitor_SMD:C_0805_2012Metric_Pad1.18x1.45mm_HandSolder, F.Cu at (-273.1, -189.0)
- added C25: 0.1u, Capacitor_SMD:C_0805_2012Metric_Pad1.18x1.45mm_HandSolder, F.Cu at (-149.9, -158.8)
- added C26: 0.1u, Capacitor_SMD:C_0805_2012Metric_Pad1.18x1.45mm_HandSolder, F.Cu at (-186.8, -166.0)
- added C27: 0.1u, Capacitor_SMD:C_0805_2012Metric_Pad1.18x1.45mm_HandSolder, F.Cu at (-202.3, -148.6)
- added C28: 0.1u, Capacitor_SMD:C_0805_2012Metric_Pad1.18x1.45mm_HandSolder, F.Cu at (-223.8, -189.2)
- added C29: 0.1u, Capacitor_SMD:C_0805_2012Metric_Pad1.18x1.45mm_HandSolder, F.Cu at (-227.3, -185.2)
- added C3: 1u, Capacitor_SMD:C_0805_2012Metric_Pad1.18x1.45mm_HandSolder, F.Cu at (69.0, -17.1)
- added C30: 0.1u, Capacitor_SMD:C_0805_2012Metric_Pad1.18x1.45mm_HandSolder, F.Cu at (-246.4, -187.7)
- added C31: 0.1u, Capacitor_SMD:C_0805_2012Metric_Pad1.18x1.45mm_HandSolder, F.Cu at (-186.8, -169.0)
- added C32: 0.1u, Capacitor_SMD:C_0805_2012Metric_Pad1.18x1.45mm_HandSolder, F.Cu at (-184.7, -177.0)
- added C33: 0.1u, Capacitor_SMD:C_0805_2012Metric_Pad1.18x1.45mm_HandSolder, F.Cu at (-194.3, -186.5)
- added C34: 0.1u, Capacitor_SMD:C_0805_2012Metric_Pad1.18x1.45mm_HandSolder, F.Cu at (-213.4, -186.9)
- added C35: 0.1u, Capacitor_SMD:C_0805_2012Metric_Pad1.18x1.45mm_HandSolder, F.Cu at (-207.1, -149.5)
- added C36: 0.1u, Capacitor_SMD:C_0805_2012Metric_Pad1.18x1.45mm_HandSolder, F.Cu at (-179.9, -177.0)
- added C37: 0.1u, Capacitor_SMD:C_0805_2012Metric_Pad1.18x1.45mm_HandSolder, F.Cu at (-80.5, -136.5)
- added C38: 4.7u, Capacitor_SMD:C_0805_2012Metric_Pad1.18x1.45mm_HandSolder, F.Cu at (-65.1, -147.8)
- added C39: 0.1u, Capacitor_SMD:C_0805_2012Metric_Pad1.18x1.45mm_HandSolder, F.Cu at (-49.7, -165.1)
- added C4: 1u, Capacitor_SMD:C_0805_2012Metric_Pad1.18x1.45mm_HandSolder, F.Cu at (73.8, -17.1)
- added C40: 4.7u, Capacitor_SMD:C_0805_2012Metric_Pad1.18x1.45mm_HandSolder, F.Cu at (-54.5, -162.1)
- added C41: 0.1u, Capacitor_SMD:C_0805_2012Metric_Pad1.18x1.45mm_HandSolder, F.Cu at (-44.8, -173.1)
- added C42: 0.1u, Capacitor_SMD:C_0805_2012Metric_Pad1.18x1.45mm_HandSolder, F.Cu at (-44.8, -170.1)
- added C43: 0.1u, Capacitor_SMD:C_0805_2012Metric_Pad1.18x1.45mm_HandSolder, F.Cu at (-37.9, -176.1)
- added C44: 0.1u, Capacitor_SMD:C_0805_2012Metric_Pad1.18x1.45mm_HandSolder, F.Cu at (-69.9, -145.6)
- added C45: 4.7u, Capacitor_SMD:C_0805_2012Metric_Pad1.18x1.45mm_HandSolder, F.Cu at (-75.7, -139.6)
- added C46: 0.1u, Capacitor_SMD:C_0805_2012Metric_Pad1.18x1.45mm_HandSolder, F.Cu at (-53.7, -159.1)
- added C47: 0.1u, Capacitor_SMD:C_0805_2012Metric_Pad1.18x1.45mm_HandSolder, F.Cu at (-47.5, -176.1)
- added C48: 0.1u, Capacitor_SMD:C_0805_2012Metric_Pad1.18x1.45mm_HandSolder, F.Cu at (-40.0, -173.1)
- added C49: 0.1u, Capacitor_SMD:C_0805_2012Metric_Pad1.18x1.45mm_HandSolder, F.Cu at (-33.1, -179.1)
- added C5: 4.7u, Capacitor_SMD:C_0805_2012Metric_Pad1.18x1.45mm_HandSolder, F.Cu at (69.0, -14.1)
- added C50: 0.1u, Capacitor_SMD:C_0805_2012Metric_Pad1.18x1.45mm_HandSolder, F.Cu at (-69.9, -142.6)
- added C51: 0.1u, Capacitor_SMD:C_0805_2012Metric_Pad1.18x1.45mm_HandSolder, F.Cu at (-75.7, -136.5)
- added C52: 0.1u, Capacitor_SMD:C_0805_2012Metric_Pad1.18x1.45mm_HandSolder, F.Cu at (-65.1, -144.8)
- added C53: 0.1u, Capacitor_SMD:C_0805_2012Metric_Pad1.18x1.45mm_HandSolder, F.Cu at (-69.9, -148.6)
- added C54: 0.1u, Capacitor_SMD:C_0805_2012Metric_Pad1.18x1.45mm_HandSolder, F.Cu at (-40.0, -170.1)
- added C55: 0.1u, Capacitor_SMD:C_0805_2012Metric_Pad1.18x1.45mm_HandSolder, F.Cu at (-37.9, -179.1)
- added C56: 0.1u, Capacitor_SMD:C_0805_2012Metric_Pad1.18x1.45mm_HandSolder, F.Cu at (-69.9, -151.6)
- added C57: 0.1u, Capacitor_SMD:C_0805_2012Metric_Pad1.18x1.45mm_HandSolder, F.Cu at (-54.5, -165.1)
- added C58: 0.1u, Capacitor_SMD:C_0805_2012Metric_Pad1.18x1.45mm_HandSolder, F.Cu at (-49.7, -168.1)
- added C59: 0.1u, Capacitor_SMD:C_0805_2012Metric_Pad1.18x1.45mm_HandSolder, F.Cu at (-42.7, -176.1)
- added C6: 4.7u, Capacitor_SMD:C_0805_2012Metric_Pad1.18x1.45mm_HandSolder, F.Cu at (45.3, -12.5)
- added C60: 0.1u, Capacitor_SMD:C_0805_2012Metric_Pad1.18x1.45mm_HandSolder, F.Cu at (-54.5, -171.1)
- added C61: 0.1u, Capacitor_SMD:C_0805_2012Metric_Pad1.18x1.45mm_HandSolder, F.Cu at (-47.5, -179.1)
- added C62: 0.1u, Capacitor_SMD:C_0805_2012Metric_Pad1.18x1.45mm_HandSolder, F.Cu at (-80.5, -139.6)
- added C63: 0.1u, Capacitor_SMD:C_0805_2012Metric_Pad1.18x1.45mm_HandSolder, F.Cu at (-49.7, -171.1)
- added C64: 0.1u, Capacitor_SMD:C_0805_2012Metric_Pad1.18x1.45mm_HandSolder, F.Cu at (-54.5, -168.1)
- added C65: 0.1u, Capacitor_SMD:C_0805_2012Metric_Pad1.18x1.45mm_HandSolder, F.Cu at (-42.7, -179.1)
- added C66: 0.1u, Capacitor_SMD:C_0805_2012Metric_Pad1.18x1.45mm_HandSolder, F.Cu at (63.0, -159.6)
- added C67: 4.7u, Capacitor_SMD:C_0805_2012Metric_Pad1.18x1.45mm_HandSolder, F.Cu at (63.0, -165.6)
- added C68: 0.1u, Capacitor_SMD:C_0805_2012Metric_Pad1.18x1.45mm_HandSolder, F.Cu at (74.7, -170.6)
- added C69: 4.7u, Capacitor_SMD:C_0805_2012Metric_Pad1.18x1.45mm_HandSolder, F.Cu at (69.9, -173.6)
- added C7: 4.7u, Capacitor_SMD:C_0805_2012Metric_Pad1.18x1.45mm_HandSolder, F.Cu at (50.1, -16.1)
- added C70: 0.1u, Capacitor_SMD:C_0805_2012Metric_Pad1.18x1.45mm_HandSolder, F.Cu at (69.9, -170.6)
- added C71: 0.1u, Capacitor_SMD:C_0805_2012Metric_Pad1.18x1.45mm_HandSolder, F.Cu at (47.5, -146.1)
- added C72: 0.1u, Capacitor_SMD:C_0805_2012Metric_Pad1.18x1.45mm_HandSolder, F.Cu at (47.5, -143.1)
- added C73: 0.1u, Capacitor_SMD:C_0805_2012Metric_Pad1.18x1.45mm_HandSolder, F.Cu at (52.3, -142.3)
- added C74: 4.7u, Capacitor_SMD:C_0805_2012Metric_Pad1.18x1.45mm_HandSolder, F.Cu at (74.7, -173.6)
- added C75: 0.1u, Capacitor_SMD:C_0805_2012Metric_Pad1.18x1.45mm_HandSolder, F.Cu at (67.8, -159.6)
- added C76: 0.1u, Capacitor_SMD:C_0805_2012Metric_Pad1.18x1.45mm_HandSolder, F.Cu at (63.7, -153.6)
- added C77: 0.1u, Capacitor_SMD:C_0805_2012Metric_Pad1.18x1.45mm_HandSolder, F.Cu at (63.0, -156.6)
- added C78: 0.1u, Capacitor_SMD:C_0805_2012Metric_Pad1.18x1.45mm_HandSolder, F.Cu at (72.6, -167.6)
- added C79: 0.1u, Capacitor_SMD:C_0805_2012Metric_Pad1.18x1.45mm_HandSolder, F.Cu at (72.6, -164.6)
- added C8: 0.1u, Capacitor_SMD:C_0805_2012Metric_Pad1.18x1.45mm_HandSolder, F.Cu at (-225.0, -151.1)
- added C80: 0.1u, Capacitor_SMD:C_0805_2012Metric_Pad1.18x1.45mm_HandSolder, F.Cu at (79.5, -170.6)
- added C81: 0.1u, Capacitor_SMD:C_0805_2012Metric_Pad1.18x1.45mm_HandSolder, F.Cu at (47.5, -140.1)
- added C82: 0.1u, Capacitor_SMD:C_0805_2012Metric_Pad1.18x1.45mm_HandSolder, F.Cu at (41.8, -134.1)
- added C83: 0.1u, Capacitor_SMD:C_0805_2012Metric_Pad1.18x1.45mm_HandSolder, F.Cu at (63.0, -162.6)
- added C84: 0.1u, Capacitor_SMD:C_0805_2012Metric_Pad1.18x1.45mm_HandSolder, F.Cu at (67.8, -165.6)
- added C85: 0.1u, Capacitor_SMD:C_0805_2012Metric_Pad1.18x1.45mm_HandSolder, F.Cu at (36.9, -134.1)
- added C86: 0.1u, Capacitor_SMD:C_0805_2012Metric_Pad1.18x1.45mm_HandSolder, F.Cu at (77.4, -167.6)
- added C87: 0.1u, Capacitor_SMD:C_0805_2012Metric_Pad1.18x1.45mm_HandSolder, F.Cu at (77.4, -164.6)
- added C88: 0.1u, Capacitor_SMD:C_0805_2012Metric_Pad1.18x1.45mm_HandSolder, F.Cu at (36.9, -131.1)
- added C89: 0.1u, Capacitor_SMD:C_0805_2012Metric_Pad1.18x1.45mm_HandSolder, F.Cu at (52.3, -139.3)
- added C9: 4.7u, Capacitor_SMD:C_0805_2012Metric_Pad1.18x1.45mm_HandSolder, F.Cu at (-207.1, -143.4)
- added C90: 0.1u, Capacitor_SMD:C_0805_2012Metric_Pad1.18x1.45mm_HandSolder, F.Cu at (79.5, -173.6)
- added C91: 0.1u, Capacitor_SMD:C_0805_2012Metric_Pad1.18x1.45mm_HandSolder, F.Cu at (41.8, -131.1)
- added C92: 0.1u, Capacitor_SMD:C_0805_2012Metric_Pad1.18x1.45mm_HandSolder, F.Cu at (47.5, -137.1)
- added C93: 0.1u, Capacitor_SMD:C_0805_2012Metric_Pad1.18x1.45mm_HandSolder, F.Cu at (67.8, -162.6)
- added C94: 0.1u, Capacitor_SMD:C_0805_2012Metric_Pad1.18x1.45mm_HandSolder, F.Cu at (84.3, -173.6)
- added D10: ESD9B3.3ST5G, Diode_SMD:D_SOD-923, F.Cu at (57.4, -7.10)
- added D11: ESD9B3.3ST5G, Diode_SMD:D_SOD-923, F.Cu at (54.7, -7.72)
- added D12: ESD9B3.3ST5G, Diode_SMD:D_SOD-923, F.Cu at (44.2, -7.10)
- added D13: RED, LED_SMD:LED_0603_1608Metric, F.Cu at (-164.0, -192.2)
- added D14: GREEN, LED_SMD:LED_0603_1608Metric, F.Cu at (-164.0, -189.7)
- added D15: RED, LED_SMD:LED_0603_1608Metric, F.Cu at (-164.0, -187.1)
- added D16: GREEN, LED_SMD:LED_0603_1608Metric, F.Cu at (-176.9, -162.3)
- added D17: RED, LED_SMD:LED_0603_1608Metric, F.Cu at (-164.0, -184.5)
- added D18: GREEN, LED_SMD:LED_0603_1608Metric, F.Cu at (-172.7, -168.3)
- added D19: RED, LED_SMD:LED_0603_1608Metric, F.Cu at (-186.5, -154.3)
- added D20: GREEN, LED_SMD:LED_0603_1608Metric, F.Cu at (-193.1, -145.9)
- added D21: RED, LED_SMD:LED_0603_1608Metric, F.Cu at (-26.8, -188.8)
- added D22: GREEN, LED_SMD:LED_0603_1608Metric, F.Cu at (-26.8, -191.4)
- added D23: RED, LED_SMD:LED_0603_1608Metric, F.Cu at (-26.8, -186.2)
- added D24: GREEN, LED_SMD:LED_0603_1608Metric, F.Cu at (-26.8, -183.6)
- added D25: RED, LED_SMD:LED_0603_1608Metric, F.Cu at (-35.6, -167.4)
- added D26: GREEN, LED_SMD:LED_0603_1608Metric, F.Cu at (-49.3, -153.5)
- added D27: RED, LED_SMD:LED_0603_1608Metric, F.Cu at (-55.9, -145.0)
- added D28: GREEN, LED_SMD:LED_0603_1608Metric, F.Cu at (-39.8, -161.4)
- added D29: RED, LED_SMD:LED_0603_1608Metric, F.Cu at (68.1, -148.0)
- added D3: ESD9B3.3ST5G, Diode_SMD:D_SOD-923, F.Cu at (49.5, -8.66)
- added D30: GREEN, LED_SMD:LED_0603_1608Metric, F.Cu at (81.8, -161.9)
- added D31: RED, LED_SMD:LED_0603_1608Metric, F.Cu at (90.6, -185.9)
- added D32: GREEN, LED_SMD:LED_0603_1608Metric, F.Cu at (90.6, -180.7)
- added D33: RED, LED_SMD:LED_0603_1608Metric, F.Cu at (90.6, -183.3)
- added D34: GREEN, LED_SMD:LED_0603_1608Metric, F.Cu at (61.5, -139.5)
- added D35: RED, LED_SMD:LED_0603_1608Metric, F.Cu at (77.7, -155.9)
- added D36: GREEN, LED_SMD:LED_0603_1608Metric, F.Cu at (90.6, -178.1)
- added D4: ESD9B3.3ST5G, Diode_SMD:D_SOD-923, F.Cu at (46.8, -6.71)
- added D5: ESD9B3.3ST5G, Diode_SMD:D_SOD-923, F.Cu at (49.5, -6.71)
- added D6: ESD9B3.3ST5G, Diode_SMD:D_SOD-923, F.Cu at (52.1, -7.72)
- added D7: ESD9B3.3ST5G, Diode_SMD:D_SOD-923, F.Cu at (63.3, -9.35)
- added D8: ESD9B3.3ST5G, Diode_SMD:D_SOD-923, F.Cu at (52.1, -5.77)
- added D9: ESD9B3.3ST5G, Diode_SMD:D_SOD-923, F.Cu at (54.7, -5.77)
- added IC3: CP2108-B03-GMR, Samacsys:QFN50P900X900X90-65N-D, F.Cu at (55.7, -149.4)
- added J1: USB_B, Connector_USB:USB_B_OST_USB-B1HSxx_Horizontal, F.Cu at (45.7, -27.7)
- added J10: DB9_Male, Connector_Dsub:DSUB-9_Male_EdgeMount_P2.77mm, F.Cu at (-198.1, -226.1)
- added J11: DB9_Male, Connector_Dsub:DSUB-9_Male_EdgeMount_P2.77mm, F.Cu at (-165.1, -226.1)
- added J12: RJ12, Connector_RJ:RJ12_Amphenol_54601, F.Cu at (-243.8, -92.7)
- added J13: RJ12, Connector_RJ:RJ12_Amphenol_54601, F.Cu at (-228.6, -92.7)
- added J14: RJ12, Connector_RJ:RJ12_Amphenol_54601, F.Cu at (-213.4, -92.7)
- added J15: RJ12, Connector_RJ:RJ12_Amphenol_54601, F.Cu at (-198.1, -92.7)
- added J16: DB9_Male, Connector_Dsub:DSUB-9_Male_EdgeMount_P2.77mm, F.Cu at (-132.1, -226.1)
- added J17: DB9_Male, Connector_Dsub:DSUB-9_Male_EdgeMount_P2.77mm, F.Cu at (-99.1, -226.1)
- added J18: DB9_Male, Connector_Dsub:DSUB-9_Male_EdgeMount_P2.77mm, F.Cu at (-66.0, -226.1)
- added J19: DB9_Male, Connector_Dsub:DSUB-9_Male_EdgeMount_P2.77mm, F.Cu at (-33.0, -226.1)
- added J2: USB_A, Connector_USB:USB_A_CONNFLY_DS1095-WNR0, F.Cu at (67.6, -32.6)
- added J20: RJ12, Connector_RJ:RJ12_Amphenol_54601, F.Cu at (-182.9, -92.7)
- added J21: RJ12, Connector_RJ:RJ12_Amphenol_54601, F.Cu at (-167.6, -92.7)
- added J22: RJ12, Connector_RJ:RJ12_Amphenol_54601, F.Cu at (-152.4, -92.7)
- added J23: RJ12, Connector_RJ:RJ12_Amphenol_54601, F.Cu at (-137.2, -92.7)
- added J24: DB9_Male, Connector_Dsub:DSUB-9_Male_EdgeMount_P2.77mm, F.Cu at (0.00, -226.1)
- added J25: DB9_Male, Connector_Dsub:DSUB-9_Male_EdgeMount_P2.77mm, F.Cu at (33.0, -226.1)
- added J26: DB9_Male, Connector_Dsub:DSUB-9_Male_EdgeMount_P2.77mm, F.Cu at (66.0, -226.1)
- added J27: DB9_Male, Connector_Dsub:DSUB-9_Male_EdgeMount_P2.77mm, F.Cu at (99.1, -226.1)
- added J3: Conn_02x20_Odd_Even, Connector_PinHeader_2.54mm:PinHeader_2x20_P2.54mm_Vertical, F.Cu at (-52.1, -53.3)
- added J4: RJ12, Connector_RJ:RJ12_Amphenol_54601, F.Cu at (-304.8, -92.7)
- added J5: RJ12, Connector_RJ:RJ12_Amphenol_54601, F.Cu at (-289.6, -92.7)
- added J6: RJ12, Connector_RJ:RJ12_Amphenol_54601, F.Cu at (-274.3, -92.7)
- added J7: RJ12, Connector_RJ:RJ12_Amphenol_54601, F.Cu at (-259.1, -92.7)
- added J8: DB9_Male, Connector_Dsub:DSUB-9_Male_EdgeMount_P2.77mm, F.Cu at (-264.2, -226.1)
- added J9: DB9_Male, Connector_Dsub:DSUB-9_Male_EdgeMount_P2.77mm, F.Cu at (-231.1, -226.1)
- added R1: 1M, Resistor_SMD:R_0805_2012Metric_Pad1.20x1.40mm_HandSolder, F.Cu at (54.8, -13.1)
- added R10: NC, Resistor_SMD:R_0805_2012Metric_Pad1.20x1.40mm_HandSolder, F.Cu at (-170.3, -177.0)
- added R11: NC, Resistor_SMD:R_0805_2012Metric_Pad1.20x1.40mm_HandSolder, F.Cu at (-172.4, -174.0)
- added R12: 0, Resistor_SMD:R_0805_2012Metric_Pad1.20x1.40mm_HandSolder, F.Cu at (-190.9, -157.0)
- added R13: 0, Resistor_SMD:R_0805_2012Metric_Pad1.20x1.40mm_HandSolder, F.Cu at (-181.3, -159.1)
- added R14: 0, Resistor_SMD:R_0805_2012Metric_Pad1.20x1.40mm_HandSolder, F.Cu at (-186.1, -160.0)
- added R15: 0, Resistor_SMD:R_0805_2012Metric_Pad1.20x1.40mm_HandSolder, F.Cu at (-165.5, -180.0)
- added R16: NC, Resistor_SMD:R_0805_2012Metric_Pad1.20x1.40mm_HandSolder, F.Cu at (-197.6, -142.6)
- added R17: NC, Resistor_SMD:R_0805_2012Metric_Pad1.20x1.40mm_HandSolder, F.Cu at (-181.3, -162.1)
- added R18: NC, Resistor_SMD:R_0805_2012Metric_Pad1.20x1.40mm_HandSolder, F.Cu at (-167.7, -174.1)
- added R19: NC, Resistor_SMD:R_0805_2012Metric_Pad1.20x1.40mm_HandSolder, F.Cu at (-165.5, -177.1)
- added R2: 56K, Resistor_SMD:R_0805_2012Metric_Pad1.20x1.40mm_HandSolder, F.Cu at (54.8, -10.2)
- added R20: 0, Resistor_SMD:R_0805_2012Metric_Pad1.20x1.40mm_HandSolder, F.Cu at (-203.3, -139.7)
- added R21: 0, Resistor_SMD:R_0805_2012Metric_Pad1.20x1.40mm_HandSolder, F.Cu at (-177.3, -165.0)
- added R22: 100, Resistor_SMD:R_0805_2012Metric_Pad1.20x1.40mm_HandSolder, F.Cu at (-192.8, -148.7)
- added R23: 100, Resistor_SMD:R_0805_2012Metric_Pad1.20x1.40mm_HandSolder, F.Cu at (-172.4, -171.0)
- added R24: 100, Resistor_SMD:R_0805_2012Metric_Pad1.20x1.40mm_HandSolder, F.Cu at (-190.9, -154.0)
- added R25: 100, Resistor_SMD:R_0805_2012Metric_Pad1.20x1.40mm_HandSolder, F.Cu at (-186.1, -157.1)
- added R26: 100, Resistor_SMD:R_0805_2012Metric_Pad1.20x1.40mm_HandSolder, F.Cu at (-197.5, -145.7)
- added R27: 100, Resistor_SMD:R_0805_2012Metric_Pad1.20x1.40mm_HandSolder, F.Cu at (-177.3, -168.0)
- added R28: 100, Resistor_SMD:R_0805_2012Metric_Pad1.20x1.40mm_HandSolder, F.Cu at (-202.3, -142.6)
- added R29: 100, Resistor_SMD:R_0805_2012Metric_Pad1.20x1.40mm_HandSolder, F.Cu at (-208.1, -137.5)
- added R3: 56K, Resistor_SMD:R_0805_2012Metric_Pad1.20x1.40mm_HandSolder, F.Cu at (59.6, -12.5)
- added R30: 0, Resistor_SMD:R_0805_2012Metric_Pad1.20x1.40mm_HandSolder, F.Cu at (-55.6, -147.8)
- added R31: 0, Resistor_SMD:R_0805_2012Metric_Pad1.20x1.40mm_HandSolder, F.Cu at (-44.9, -167.1)
- added R32: 1K, Resistor_SMD:R_0805_2012Metric_Pad1.20x1.40mm_HandSolder, F.Cu at (-49.7, -162.1)
- added R33: NC, Resistor_SMD:R_0805_2012Metric_Pad1.20x1.40mm_HandSolder, F.Cu at (-60.3, -147.8)
- added R34: NC, Resistor_SMD:R_0805_2012Metric_Pad1.20x1.40mm_HandSolder, F.Cu at (-44.9, -164.2)
- added R35: NC, Resistor_SMD:R_0805_2012Metric_Pad1.20x1.40mm_HandSolder, F.Cu at (-33.1, -176.1)
- added R36: NC, Resistor_SMD:R_0805_2012Metric_Pad1.20x1.40mm_HandSolder, F.Cu at (-44.2, -158.3)
- added R37: 0, Resistor_SMD:R_0805_2012Metric_Pad1.20x1.40mm_HandSolder, F.Cu at (-35.3, -173.1)
- added R38: 0, Resistor_SMD:R_0805_2012Metric_Pad1.20x1.40mm_HandSolder, F.Cu at (-60.4, -141.8)
- added R39: 0, Resistor_SMD:R_0805_2012Metric_Pad1.20x1.40mm_HandSolder, F.Cu at (-44.2, -161.2)
- added R4: 12k, Resistor_SMD:R_0805_2012Metric_Pad1.20x1.40mm_HandSolder, F.Cu at (59.6, -9.55)
- added R40: 0, Resistor_SMD:R_0805_2012Metric_Pad1.20x1.40mm_HandSolder, F.Cu at (-30.5, -173.2)
- added R41: NC, Resistor_SMD:R_0805_2012Metric_Pad1.20x1.40mm_HandSolder, F.Cu at (-28.3, -176.2)
- added R42: NC, Resistor_SMD:R_0805_2012Metric_Pad1.20x1.40mm_HandSolder, F.Cu at (-66.1, -138.8)
- added R43: NC, Resistor_SMD:R_0805_2012Metric_Pad1.20x1.40mm_HandSolder, F.Cu at (-40.1, -164.2)
- added R44: NC, Resistor_SMD:R_0805_2012Metric_Pad1.20x1.40mm_HandSolder, F.Cu at (-53.7, -156.1)
- added R45: 0, Resistor_SMD:R_0805_2012Metric_Pad1.20x1.40mm_HandSolder, F.Cu at (-35.3, -170.2)
- added R46: 0, Resistor_SMD:R_0805_2012Metric_Pad1.20x1.40mm_HandSolder, F.Cu at (-70.9, -139.6)
- added R47: 100, Resistor_SMD:R_0805_2012Metric_Pad1.20x1.40mm_HandSolder, F.Cu at (-53.7, -153.2)
- added R48: 100, Resistor_SMD:R_0805_2012Metric_Pad1.20x1.40mm_HandSolder, F.Cu at (-48.9, -156.2)
- added R49: 100, Resistor_SMD:R_0805_2012Metric_Pad1.20x1.40mm_HandSolder, F.Cu at (-60.3, -144.9)
- added R5: 0, Resistor_SMD:R_0805_2012Metric_Pad1.20x1.40mm_HandSolder, F.Cu at (-208.1, -140.4)
- added R50: 100, Resistor_SMD:R_0805_2012Metric_Pad1.20x1.40mm_HandSolder, F.Cu at (-40.1, -167.1)
- added R51: 100, Resistor_SMD:R_0805_2012Metric_Pad1.20x1.40mm_HandSolder, F.Cu at (-65.2, -141.8)
- added R52: 100, Resistor_SMD:R_0805_2012Metric_Pad1.20x1.40mm_HandSolder, F.Cu at (-70.9, -136.6)
- added R53: 100, Resistor_SMD:R_0805_2012Metric_Pad1.20x1.40mm_HandSolder, F.Cu at (-28.3, -179.2)
- added R54: 100, Resistor_SMD:R_0805_2012Metric_Pad1.20x1.40mm_HandSolder, F.Cu at (-48.9, -159.2)
- added R55: 0, Resistor_SMD:R_0805_2012Metric_Pad1.20x1.40mm_HandSolder, F.Cu at (72.6, -161.6)
- added R56: 0, Resistor_SMD:R_0805_2012Metric_Pad1.20x1.40mm_HandSolder, F.Cu at (46.5, -134.1)
- added R57: 1K, Resistor_SMD:R_0805_2012Metric_Pad1.20x1.40mm_HandSolder, F.Cu at (57.1, -142.3)
- added R58: NC, Resistor_SMD:R_0805_2012Metric_Pad1.20x1.40mm_HandSolder, F.Cu at (82.2, -164.7)
- added R59: NC, Resistor_SMD:R_0805_2012Metric_Pad1.20x1.40mm_HandSolder, F.Cu at (72.6, -158.7)
- added R6: 0, Resistor_SMD:R_0805_2012Metric_Pad1.20x1.40mm_HandSolder, F.Cu at (-182.0, -168.0)
- added R60: NC, Resistor_SMD:R_0805_2012Metric_Pad1.20x1.40mm_HandSolder, F.Cu at (63.7, -147.7)
- added R61: NC, Resistor_SMD:R_0805_2012Metric_Pad1.20x1.40mm_HandSolder, F.Cu at (68.5, -150.7)
- added R62: 0, Resistor_SMD:R_0805_2012Metric_Pad1.20x1.40mm_HandSolder, F.Cu at (57.1, -139.4)
- added R63: 0, Resistor_SMD:R_0805_2012Metric_Pad1.20x1.40mm_HandSolder, F.Cu at (77.3, -161.6)
- added R64: 0, Resistor_SMD:R_0805_2012Metric_Pad1.20x1.40mm_HandSolder, F.Cu at (52.3, -136.3)
- added R65: 0, Resistor_SMD:R_0805_2012Metric_Pad1.20x1.40mm_HandSolder, F.Cu at (46.5, -131.1)
- added R66: NC, Resistor_SMD:R_0805_2012Metric_Pad1.20x1.40mm_HandSolder, F.Cu at (89.1, -173.7)
- added R67: NC, Resistor_SMD:R_0805_2012Metric_Pad1.20x1.40mm_HandSolder, F.Cu at (68.5, -153.7)
- added R68: NC, Resistor_SMD:R_0805_2012Metric_Pad1.20x1.40mm_HandSolder, F.Cu at (63.7, -150.6)
- added R69: NC, Resistor_SMD:R_0805_2012Metric_Pad1.20x1.40mm_HandSolder, F.Cu at (82.2, -167.6)
- added R7: 1K, Resistor_SMD:R_0805_2012Metric_Pad1.20x1.40mm_HandSolder, F.Cu at (-186.8, -163.0)
- added R70: 0, Resistor_SMD:R_0805_2012Metric_Pad1.20x1.40mm_HandSolder, F.Cu at (73.2, -152.8)
- added R71: 0, Resistor_SMD:R_0805_2012Metric_Pad1.20x1.40mm_HandSolder, F.Cu at (67.7, -156.6)
- added R72: 100, Resistor_SMD:R_0805_2012Metric_Pad1.20x1.40mm_HandSolder, F.Cu at (61.8, -142.3)
- added R73: 100, Resistor_SMD:R_0805_2012Metric_Pad1.20x1.40mm_HandSolder, F.Cu at (57.0, -136.3)
- added R74: 100, Resistor_SMD:R_0805_2012Metric_Pad1.20x1.40mm_HandSolder, F.Cu at (73.2, -155.7)
- added R75: 100, Resistor_SMD:R_0805_2012Metric_Pad1.20x1.40mm_HandSolder, F.Cu at (86.9, -167.7)
- added R76: 100, Resistor_SMD:R_0805_2012Metric_Pad1.20x1.40mm_HandSolder, F.Cu at (89.1, -170.7)
- added R77: 100, Resistor_SMD:R_0805_2012Metric_Pad1.20x1.40mm_HandSolder, F.Cu at (51.3, -133.3)
- added R78: 100, Resistor_SMD:R_0805_2012Metric_Pad1.20x1.40mm_HandSolder, F.Cu at (77.3, -158.7)
- added R79: 100, Resistor_SMD:R_0805_2012Metric_Pad1.20x1.40mm_HandSolder, F.Cu at (84.3, -170.7)
- added R8: NC, Resistor_SMD:R_0805_2012Metric_Pad1.20x1.40mm_HandSolder, F.Cu at (-197.5, -148.7)
- added R9: NC, Resistor_SMD:R_0805_2012Metric_Pad1.20x1.40mm_HandSolder, F.Cu at (-182.0, -165.0)
- added U10: SP3243, Package_SO:SSOP-28_5.3x10.2mm_P0.65mm, F.Cu at (-73.7, -171.4)
- added U11: SP3243, Package_SO:SSOP-28_5.3x10.2mm_P0.65mm, F.Cu at (29.2, -184.2)
- added U12: SP3243, Package_SO:SSOP-28_5.3x10.2mm_P0.65mm, F.Cu at (43.2, -184.2)
- added U13: SP3243, Package_SO:SSOP-28_5.3x10.2mm_P0.65mm, F.Cu at (57.1, -184.2)
- added U14: SP3243, Package_SO:SSOP-28_5.3x10.2mm_P0.65mm, F.Cu at (71.1, -184.2)
- added U3: SP3243, Package_SO:SSOP-28_5.3x10.2mm_P0.65mm, F.Cu at (-248.9, -163.8)
- added U4: SP3243, Package_SO:SSOP-28_5.3x10.2mm_P0.65mm, F.Cu at (-261.6, -185.4)
- added U5: SP3243, Package_SO:SSOP-28_5.3x10.2mm_P0.65mm, F.Cu at (-236.2, -182.9)
- added U6: SP3243, Package_SO:SSOP-28_5.3x10.2mm_P0.65mm, F.Cu at (-204.5, -182.9)
- added U7: SP3243, Package_SO:SSOP-28_5.3x10.2mm_P0.65mm, F.Cu at (-123.2, -171.4)
- added U8: SP3243, Package_SO:SSOP-28_5.3x10.2mm_P0.65mm, F.Cu at (-105.4, -171.4)
- added U9: SP3243, Package_SO:SSOP-28_5.3x10.2mm_P0.65mm, F.Cu at (-88.9, -171.4)
- added Y1: 24M, Crystal:Crystal_SMD_2016-4Pin_2.0x1.6mm, F.Cu at (63.9, -12.2)
- D1, D2: value SP0503BAHT -> ESD9B3.3ST5G; footprint Package_TO_SOT_SMD:SOT-143 -> Diode_SMD:D_SOD-923
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Connections:
- D1 pad 1: GND -> /VBUS_5V
- D1 pad 2: /VBUS_5V -> GND
- D2 pad 1: GND -> /D+_UPSTREAM
- D2 pad 2: /VBUS_5V -> GND
- IC1 pad 1: Net-(IC1-Pad1) -> /2108_Block A/RXD4
- IC1 pad 10: Net-(IC1-Pad10) -> /2108_Block A/DTR4
- IC1 pad 11: Net-(IC1-Pad11) -> /2108_Block A/RI3
- IC1 pad 12: Net-(IC1-Pad12) -> /2108_Block A/DCD3
- IC1 pad 13: Net-(IC1-Pad13) -> /2108_Block A/CTS3
- IC1 pad 14: Net-(IC1-Pad14) -> /2108_Block A/RTS3
- IC1 pad 15: Net-(IC1-Pad15) -> /2108_Block A/RXD3
- IC1 pad 16: Net-(IC1-Pad16) -> /2108_Block A/TXD3
- IC1 pad 17: Net-(IC1-Pad17) -> /2108_Block A/DSR3
- IC1 pad 18: Net-(IC1-Pad18) -> /2108_Block A/DTR3
- IC1 pad 19: Net-(IC1-Pad19) -> /2108_Block A/~SUSPEND
- IC1 pad 2: Net-(IC1-Pad2) -> GND
- IC1 pad 21: Net-(IC1-Pad21) -> /IO8
- IC1 pad 22: Net-(IC1-Pad22) -> /IO7
- IC1 pad 23: Net-(IC1-Pad23) -> /2108_Block A/RXD3_LED
- IC1 pad 24: Net-(IC1-Pad24) -> /2108_Block A/3V3_NET
- IC1 pad 25: Net-(IC1-Pad25) -> GND
- IC1 pad 26: Net-(IC1-Pad26) -> /2108_Block A/TXD3_LED
- IC1 pad 27: Net-(IC1-Pad27) -> /IO6
- IC1 pad 28: Net-(IC1-Pad28) -> /IO5
- IC1 pad 29: Net-(IC1-Pad29) -> /2108_Block A/RXD3_LED
- IC1 pad 3: Net-(IC1-Pad3) -> /2108_Block A/3V3_NET
- IC1 pad 30: Net-(IC1-Pad30) -> /2108_Block A/TXD3_LED
- IC1 pad 31: Net-(IC1-Pad31) -> /IO4
- IC1 pad 32: Net-(IC1-Pad32) -> /IO3
- IC1 pad 33: Net-(IC1-Pad33) -> /2108_Block A/RXD2_LED
- IC1 pad 34: Net-(IC1-Pad34) -> /2108_Block A/TXD2_LED
- IC1 pad 37: Net-(IC1-Pad37) -> /IO2
- IC1 pad 38: Net-(IC1-Pad38) -> /IO1
- IC1 pad 39: Net-(IC1-Pad39) -> /2108_Block A/3V3_NET
- IC1 pad 4: Net-(IC1-Pad4) -> /2108_Block A/TXD4
- IC1 pad 40: Net-(IC1-Pad40) -> /2108_Block A/RXD1_LED
- IC1 pad 41: Net-(IC1-Pad41) -> /2108_Block A/TXD1_LED
- IC1 pad 42: Net-(IC1-Pad42) -> /2108_Block A/RI2
- IC1 pad 43: Net-(IC1-Pad43) -> /2108_Block A/DCD2
- IC1 pad 44: Net-(IC1-Pad44) -> /2108_Block A/DSR2
- IC1 pad 45: Net-(IC1-Pad45) -> /2108_Block A/DTR2
- IC1 pad 46: Net-(IC1-Pad46) -> /2108_Block A/CTS2
- IC1 pad 47: Net-(IC1-Pad47) -> /2108_Block A/RTS2
- IC1 pad 48: Net-(IC1-Pad48) -> /2108_Block A/RXD2
- IC1 pad 49: Net-(IC1-Pad49) -> /2108_Block A/TXD2
- IC1 pad 5: Net-(IC1-Pad5) -> /2108_Block A/CTS4
- IC1 pad 50: Net-(IC1-Pad50) -> /2108_Block A/RI1
- IC1 pad 51: Net-(IC1-Pad51) -> /2108_Block A/DCD1
- IC1 pad 52: Net-(IC1-Pad52) -> /2108_Block A/DSR1
- IC1 pad 53: Net-(IC1-Pad53) -> /2108_Block A/DTR1
- IC1 pad 54: Net-(IC1-Pad54) -> /2108_Block A/CTS1
- IC1 pad 55: Net-(IC1-Pad55) -> /2108_Block A/RTS1
- IC1 pad 56: Net-(IC1-Pad56) -> /2108_Block A/RXD1
- IC1 pad 57: Net-(IC1-Pad57) -> /2108_Block A/TXD1
- IC1 pad 58: Net-(IC1-Pad58) -> /2108_Block A/3V3_NET
- IC1 pad 59: Net-(IC1-Pad59) -> GND
- IC1 pad 6: Net-(IC1-Pad6) -> /2108_Block A/RTS4
- IC1 pad 60: Net-(IC1-Pad60) -> /VBUS_5V
- IC1 pad 61: Net-(IC1-Pad61) -> /VBUS_5V
- IC1 pad 62: Net-(IC1-Pad62) -> /D+_1
- IC1 pad 63: Net-(IC1-Pad63) -> /D-_1
- IC1 pad 65: Net-(IC1-Pad65) -> GND
- IC1 pad 7: Net-(IC1-Pad7) -> /2108_Block A/RI4
- IC1 pad 8: Net-(IC1-Pad8) -> /2108_Block A/DCD4
- IC1 pad 9: Net-(IC1-Pad9) -> /2108_Block A/DSR4
- IC2 pad 1: Net-(IC2-Pad1) -> /2108_Block B/RXD4
- IC2 pad 10: Net-(IC2-Pad10) -> /2108_Block B/DTR4
- IC2 pad 11: Net-(IC2-Pad11) -> /2108_Block B/RI3
- IC2 pad 12: Net-(IC2-Pad12) -> /2108_Block B/DCD3
- IC2 pad 13: Net-(IC2-Pad13) -> /2108_Block B/CTS3
- IC2 pad 14: Net-(IC2-Pad14) -> /2108_Block B/RTS3
- IC2 pad 15: Net-(IC2-Pad15) -> /2108_Block B/RXD3
- IC2 pad 16: Net-(IC2-Pad16) -> /2108_Block B/TXD3
- IC2 pad 17: Net-(IC2-Pad17) -> /2108_Block B/DSR3
- IC2 pad 18: Net-(IC2-Pad18) -> /2108_Block B/DTR3
- IC2 pad 19: Net-(IC2-Pad19) -> /2108_Block B/~SUSPEND
- IC2 pad 2: Net-(IC2-Pad2) -> GND
- IC2 pad 21: Net-(IC2-Pad21) -> /IO16
- IC2 pad 22: Net-(IC2-Pad22) -> /IO15
- IC2 pad 23: Net-(IC2-Pad23) -> /2108_Block B/RXD3_LED
- IC2 pad 24: Net-(IC2-Pad24) -> /2108_Block B/3V3_NET
- IC2 pad 25: Net-(IC2-Pad25) -> GND
- IC2 pad 26: Net-(IC2-Pad26) -> /2108_Block B/TXD3_LED
- IC2 pad 27: Net-(IC2-Pad27) -> /IO14
- IC2 pad 28: Net-(IC2-Pad28) -> /IO13
- IC2 pad 29: Net-(IC2-Pad29) -> /2108_Block B/RXD3_LED
- IC2 pad 3: Net-(IC2-Pad3) -> /2108_Block B/3V3_NET
- IC2 pad 30: Net-(IC2-Pad30) -> /2108_Block B/TXD3_LED
- IC2 pad 31: Net-(IC2-Pad31) -> /IO12
- IC2 pad 32: Net-(IC2-Pad32) -> /IO11
- IC2 pad 33: Net-(IC2-Pad33) -> /2108_Block B/RXD2_LED
- IC2 pad 34: Net-(IC2-Pad34) -> /2108_Block B/TXD2_LED
- IC2 pad 37: Net-(IC2-Pad37) -> /IO10
- IC2 pad 38: Net-(IC2-Pad38) -> /IO9
- IC2 pad 39: Net-(IC2-Pad39) -> /2108_Block B/3V3_NET
- IC2 pad 4: Net-(IC2-Pad4) -> /2108_Block B/TXD4
- IC2 pad 40: Net-(IC2-Pad40) -> /2108_Block B/RXD1_LED
- IC2 pad 41: Net-(IC2-Pad41) -> /2108_Block B/TXD1_LED
- IC2 pad 42: Net-(IC2-Pad42) -> /2108_Block B/RI2
- IC2 pad 43: Net-(IC2-Pad43) -> /2108_Block B/DCD2
- IC2 pad 44: Net-(IC2-Pad44) -> /2108_Block B/DSR2
- IC2 pad 45: Net-(IC2-Pad45) -> /2108_Block B/DTR2
- IC2 pad 46: Net-(IC2-Pad46) -> /2108_Block B/CTS2
- IC2 pad 47: Net-(IC2-Pad47) -> /2108_Block B/RTS2
- IC2 pad 48: Net-(IC2-Pad48) -> /2108_Block B/RXD2
- IC2 pad 49: Net-(IC2-Pad49) -> /2108_Block B/TXD2
- IC2 pad 5: Net-(IC2-Pad5) -> /2108_Block B/CTS4
- IC2 pad 50: Net-(IC2-Pad50) -> /2108_Block B/RI1
- IC2 pad 51: Net-(IC2-Pad51) -> /2108_Block B/DCD1
- IC2 pad 52: Net-(IC2-Pad52) -> /2108_Block B/DSR1
- IC2 pad 53: Net-(IC2-Pad53) -> /2108_Block B/DTR1
- IC2 pad 54: Net-(IC2-Pad54) -> /2108_Block B/CTS1
- IC2 pad 55: Net-(IC2-Pad55) -> /2108_Block B/RTS1
- IC2 pad 56: Net-(IC2-Pad56) -> /2108_Block B/RXD1
- IC2 pad 57: Net-(IC2-Pad57) -> /2108_Block B/TXD1
- IC2 pad 58: Net-(IC2-Pad58) -> /2108_Block B/3V3_NET
- IC2 pad 59: Net-(IC2-Pad59) -> GND
- IC2 pad 6: Net-(IC2-Pad6) -> /2108_Block B/RTS4
- IC2 pad 60: Net-(IC2-Pad60) -> /VBUS_5V
- IC2 pad 61: Net-(IC2-Pad61) -> /VBUS_5V
- IC2 pad 62: Net-(IC2-Pad62) -> /D+_2
- IC2 pad 63: Net-(IC2-Pad63) -> /D-_2
- IC2 pad 65: Net-(IC2-Pad65) -> GND
- IC2 pad 7: Net-(IC2-Pad7) -> /2108_Block B/RI4
- IC2 pad 8: Net-(IC2-Pad8) -> /2108_Block B/DCD4
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
Commit message: Netlist #2
Parts:
- C1, C2: value 18p -> 6p
- R22, R23, R24, R25, R26, R27, R28, R29, R47, R48, R49, R50, R51, R52, R53, R54, R72, R73, R74, R75, R76, R77, R78, R79: value 100 -> 270
- moved D31 270.9 mm to (-165.5, -97.4), turned to 90 degrees
- moved D30 268.3 mm to (-178.6, -97.4), turned to 90 degrees
- moved D32 267.3 mm to (-163.4, -97.4), turned to 90 degrees
- moved R75 259.0 mm to (-163.4, -101.0), turned to 270 degrees
- moved D33 255.7 mm to (-150.2, -97.4), turned to 90 degrees
- moved D29 253.8 mm to (-180.6, -97.4), turned to 90 degrees
- moved R76 249.3 mm to (-150.2, -101.0), turned to 270 degrees
- moved R72 246.0 mm to (-180.6, -101.0), turned to 270 degrees
- moved R74 244.9 mm to (-165.5, -101.0), turned to 270 degrees
- moved R73 238.2 mm to (-178.6, -101.0), turned to 270 degrees
- moved D36 237.6 mm to (-132.9, -97.4), turned to 90 degrees
- moved D21 233.5 mm to (-241.7, -97.4), turned to 90 degrees
- moved D22 232.6 mm to (-239.6, -97.4), turned to 90 degrees
- moved R79 228.1 mm to (-132.9, -101.0), turned to 270 degrees
- moved D35 220.5 mm to (-135.0, -97.4), turned to 90 degrees
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
Commit message: Layout in prgs. 1
Parts:
- moved R58 267.5 mm to (-178.6, -105.1), turned to 270 degrees
- moved R55 255.4 mm to (-176.5, -105.1), turned to 270 degrees
- moved R63 251.3 mm to (-167.5, -105.1), turned to 270 degrees
- moved R60 248.0 mm to (-180.6, -105.1), turned to 270 degrees
- moved R66 246.9 mm to (-148.1, -105.1), turned to 270 degrees
- moved R62 242.2 mm to (-182.7, -105.1), turned to 270 degrees
- moved R59 241.9 mm to (-163.4, -105.1), turned to 270 degrees
- moved R61 238.4 mm to (-165.5, -105.1), turned to 270 degrees
- moved R70 230.5 mm to (-152.3, -105.1), turned to 270 degrees
- moved R69 226.0 mm to (-135.0, -105.1), turned to 270 degrees
- moved R35 220.3 mm to (-241.7, -105.1), turned to 270 degrees
- moved R37 219.3 mm to (-243.7, -105.1), turned to 270 degrees
- moved R68 218.7 mm to (-150.2, -105.1), turned to 270 degrees
- moved R71 211.2 mm to (-137.1, -105.1), turned to 270 degrees
- moved R56 209.8 mm to (-161.3, -105.1), turned to 270 degrees
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
Commit message: Layout in prgs. 2
Parts:
- moved C68 191.8 mm to (-83.7, -278.9), turned to 180 degrees
- moved C66 190.0 mm to (-88.1, -274.7)
- moved C73 189.8 mm to (-83.7, -274.7), turned to 180 degrees
- moved C70 188.9 mm to (-92.6, -267.1)
- moved C74 186.8 mm to (-83.7, -272.6), turned to 180 degrees
- moved C67 185.2 mm to (-88.1, -272.6)
- moved C69 185.0 mm to (-83.7, -276.8), turned to 180 degrees
- moved IC3 180.8 mm to (-84.0, -264.3)
- moved C72 172.2 mm to (-75.6, -263.6), turned to 180 degrees
- moved C71 171.6 mm to (-84.2, -256.1), turned to 90 degrees
- moved C37 138.4 mm to (-88.1, -274.7)
- moved C45 133.3 mm to (-83.7, -272.6), turned to 180 degrees
- moved C44 129.9 mm to (-83.7, -274.7), turned to 180 degrees
- moved C9 129.8 mm to (-219.4, -272.6)
- moved C38 127.0 mm to (-88.1, -272.6)
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
Commit message: layout in prgs
Parts:
- J10, J11, J16, J17, J18, J19, J24, J25, J26, J27, J8, J9: footprint Connector_Dsub:DSUB-9_Male_EdgeMount_P2.77mm -> Connector_Dsub:DSUB-9_Male_Vertical_P2.77x2.84mm
- J12, J13, J14, J15, J20, J21, J22, J23, J4, J5, J6, J7: value RJ12 -> RJ25; footprint Connector_RJ:RJ12_Amphenol_54601 -> Connector_RJ:RJ25_Wayconn_MJEA-660X1_Horizontal
- R5: moved to B.Cu
- R7: renamed from R8; moved to B.Cu
- R8: renamed from R10; moved to B.Cu
- R9: renamed from R12; moved to B.Cu
- moved C17 111.9 mm to (-356.6, -183.8)
- moved J8 110.7 mm to (-353.7, -161.0), turned to 90 degrees
- moved C19 110.6 mm to (-355.3, -199.4), turned to 180 degrees
- moved C18 108.8 mm to (-357.3, -197.0), turned to 180 degrees
- moved C25 108.1 mm to (-353.4, -197.0), turned to 180 degrees
- moved C20 107.5 mm to (-358.6, -187.0)
- moved U3 102.6 mm to (-351.9, -190.5), turned to 90 degrees
- moved C21 95.8 mm to (-273.1, -162.0)
- moved C24 90.4 mm to (-275.2, -165.2)
- moved C22 86.2 mm to (-273.8, -175.2), turned to 180 degrees
- moved C26 84.2 mm to (-269.9, -175.2), turned to 180 degrees
- moved C23 83.7 mm to (-271.9, -177.6), turned to 180 degrees
- moved U4 82.8 mm to (-268.5, -168.7), turned to 90 degrees
- moved J9 75.5 mm to (-242.0, -151.3), turned to 90 degrees
- moved D13 69.9 mm to (-353.5, -145.4), turned to 270 degrees
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- renumbered R14 to R10, R16 to R11, R18 to R12, R20 to R13, R6 to R14, R9 to R15, R11 to R16, R13 to R17, R15 to R18, R17 to R19, R19 to R20, R32 to R31, R33 to R32, R35 to R33, R37 to R34, R39 to R35, R41 to R36, R43 to R37, R45 to R38, R31 to R39, R34 to R40, R36 to R41, R38 to R42, R40 to R43, R42 to R44, R44 to R45, R57 to R56, R58 to R57, R60 to R58, R62 to R59, R7 to R6, R64 to R60, R66 to R61, R68 to R62, R70 to R63, R56 to R64, R59 to R65, R61 to R66, R63 to R67, R65 to R68, R67 to R69, R69 to R70
Connections:
- R10 pad 2: Net-(J6-Pad5) -> Net-(J5-Pad5)
- R11 pad 2: Net-(J6-Pad5) -> Net-(J5-Pad5)
- R12 pad 2: Net-(J6-Pad2) -> Net-(J5-Pad2)
- R13 pad 2: Net-(J6-Pad2) -> Net-(J5-Pad2)
- R14 pad 2: Net-(J5-Pad5) -> Net-(J6-Pad5)
- R15 pad 2: Net-(J5-Pad5) -> Net-(J6-Pad5)
- R16 pad 2: Net-(J5-Pad2) -> Net-(J6-Pad2)
- R17 pad 2: Net-(J5-Pad2) -> Net-(J6-Pad2)
- R35 pad 2: Net-(J14-Pad5) -> Net-(J13-Pad5)
- R36 pad 2: Net-(J14-Pad5) -> Net-(J13-Pad5)
- R37 pad 2: Net-(J14-Pad2) -> Net-(J13-Pad2)
- R38 pad 2: Net-(J14-Pad2) -> Net-(J13-Pad2)
- R39 pad 2: Net-(J13-Pad5) -> Net-(J14-Pad5)
- R40 pad 2: Net-(J13-Pad5) -> Net-(J14-Pad5)
- R41 pad 2: Net-(J13-Pad2) -> Net-(J14-Pad2)
- R42 pad 2: Net-(J13-Pad2) -> Net-(J14-Pad2)
- R60 pad 2: Net-(J22-Pad5) -> Net-(J21-Pad5)
- R61 pad 2: Net-(J22-Pad5) -> Net-(J21-Pad5)
- R62 pad 2: Net-(J22-Pad2) -> Net-(J21-Pad2)
- R63 pad 2: Net-(J22-Pad2) -> Net-(J21-Pad2)
- R64 pad 2: Net-(J21-Pad5) -> Net-(J22-Pad5)
- R65 pad 2: Net-(J21-Pad5) -> Net-(J22-Pad5)
- R66 pad 2: Net-(J21-Pad2) -> Net-(J22-Pad2)
- R67 pad 2: Net-(J21-Pad2) -> Net-(J22-Pad2)
Routing:
- net /2108_Block A/TXD232_1: track 0.00 -> 53.5 mm, vias 0 -> 1
- net /2108_Block A/RXD232_1: track 0.00 -> 48.0 mm
- net /2108_Block A/3V3_NET: track 0.00 -> 33.0 mm, vias 0 -> 4
- net /2108_Block A/DCD232_1: track 0.00 -> 30.7 mm
- net /2108_Block A/RXD232_2: track 0.00 -> 28.8 mm
- net /2108_Block A/DSR232_1: track 0.00 -> 26.3 mm
- net /2108_Block A/RTS232_1: track 0.00 -> 24.2 mm, vias 0 -> 1
- net /2108_Block A/DTR232_1: track 0.00 -> 23.8 mm, vias 0 -> 1
- net Net-(J7-Pad2): track 0.00 -> 22.9 mm
- net /2108_Block A/CTS232_1: track 0.00 -> 20.1 mm
- net /2108_Block A/RI232_1: track 0.00 -> 16.5 mm, vias 0 -> 2
- net Net-(J7-Pad5): track 0.00 -> 14.0 mm
- net Net-(J4-Pad2): track 0.00 -> 10.8 mm
- net Net-(J4-Pad5): track 0.00 -> 6.77 mm
- net Net-(J5-Pad2): track 0.00 -> 6.31 mm
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
Commit message: layout in prgs
Parts:
- C10, C11, C19, C23, C29, C33, C48, C52, C58, C62, C77, C81, C87, C91, R10, R11, R12, R13, R14, R15, R16, R17, R18, R19, R20, R21, R30, R32, R33, R34, R35, R36, R37, R38, R39, R40, R41, R42, R43, R44, R45, R46, R55, R57, R58, R59, R60, R61, R62, R63, R64, R65, R66, R67, R68, R69, R70, R71: moved to B.Cu
- moved C19 500.6 mm to (60.0, 80.0)
- moved C18 494.9 mm to (57.3, 73.3)
- moved C25 494.9 mm to (61.3, 73.3)
- moved U3 494.9 mm to (62.7, 79.8)
- moved C20 494.3 mm to (55.9, 82.3), turned to 270 degrees
- moved J8 494.2 mm to (59.7, 109.8)
- moved C17 494.2 mm to (57.7, 85.7)
- moved J4 493.7 mm to (63.7, 129.8)
- moved D13 493.5 mm to (60.0, 123.9)
- moved D14 493.5 mm to (62.2, 123.9)
- moved R22 493.5 mm to (58.0, 124.2)
- moved R23 493.5 mm to (64.2, 124.2)
- moved R5 493.5 mm to (59.6, 123.8)
- moved R7 493.5 mm to (57.5, 123.8)
- moved R8 493.5 mm to (64.7, 123.8)
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Routing:
- net /2108_Block A/TXD232_1: track 53.5 -> 0.00 mm, vias 1 -> 0
- net /2108_Block A/RXD232_1: track 48.0 -> 0.00 mm
- net /2108_Block A/DCD232_1: track 30.7 -> 0.00 mm
- net /2108_Block A/RXD232_2: track 28.8 -> 0.00 mm
- net /2108_Block A/DSR232_1: track 26.3 -> 0.00 mm
- net /2108_Block A/RTS232_1: track 24.2 -> 0.00 mm, vias 1 -> 0
- net /2108_Block A/DTR232_1: track 23.8 -> 0.00 mm, vias 1 -> 0
- net Net-(J7-Pad2): track 22.9 -> 0.00 mm
- net /2108_Block A/CTS232_1: track 20.1 -> 0.00 mm
- net /2108_Block A/RI232_1: track 16.5 -> 0.00 mm, vias 2 -> 0
- net /2108_Block A/3V3_NET: track 33.0 -> 18.0 mm, vias 4 -> 0
- net Net-(J7-Pad5): track 14.0 -> 0.00 mm
- net Net-(J4-Pad2): track 10.8 -> 0.00 mm
- net /VBUS_5V: track 0.00 -> 7.61 mm
- net Net-(J4-Pad5): track 6.77 -> 0.00 mm
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
Commit message: PCB layout in prgs.
Parts:
- J10, J11, J16, J17, J18, J19, J24, J25, J26, J27, J8, J9: footprint Connector_Dsub:DSUB-9_Male_Vertical_P2.77x2.84mm -> Connector_Dsub:DSUB-9_Male_Vertical_P2.77x2.84mm_MountingHoles
- moved R31 196.9 mm to (96.4, -30.0)
- moved R56 196.9 mm to (203.1, -10.2)
- moved IC2 75.1 mm to (149.9, 63.5)
- moved C8 57.2 mm to (25.3, 25.2)
- moved C9 57.2 mm to (25.3, 27.3)
- moved C10 57.2 mm to (30.8, 27.3)
- moved C11 57.2 mm to (30.8, 25.2)
- moved C15 57.2 mm to (30.8, 25.2)
- moved C16 57.2 mm to (30.8, 27.3)
- moved C14 54.6 mm to (37.6, 52.9)
- moved C13 54.6 mm to (28.9, 60.3)
- moved C12 52.6 mm to (25.1, 34.5), turned to 90 degrees
- moved C41 43.2 mm to (234.3, 3.64)
- moved C42 43.2 mm to (242.6, 14.6)
- moved C70 43.2 mm to (234.3, 3.64)
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Connections:
- net /D+_1 renamed /D_1_P
- net /D+_2 renamed /D_2_P
- net /D+_3 renamed /D_3_P
- net /D+_4 renamed /D_4_P
- net /D+_UPSTREAM renamed /D_UPSTREAM_P
- net /D-_1 renamed /D_1_N
- net /D-_2 renamed /D_2_N
- net /D-_3 renamed /D_3_N
- net /D-_4 renamed /D_4_N
- net /D-_UPSTREAM renamed /D_UPSTREAM_N
Routing:
- net /D_3_P: track 0.00 -> 115.8 mm
- net /D_3_N: track 0.00 -> 115.8 mm
- net /2108_Block A/RXD232_3: track 0.00 -> 115.0 mm
- net /2108_Block A/TXD232_3: track 0.00 -> 111.8 mm, vias 0 -> 4
- net /2108_Block A/DSR232_3: track 0.00 -> 68.2 mm
- net /2108_Block A/DCD232_3: track 0.00 -> 64.7 mm, vias 0 -> 2
- net /2108_Block A/CTS232_3: track 0.00 -> 59.6 mm, vias 0 -> 2
- net /2108_Block A/RXD232_1: track 0.00 -> 57.7 mm
- net /2108_Block A/TXD232_1: track 0.00 -> 55.9 mm, vias 0 -> 2
- net /D_2_P: track 0.00 -> 51.1 mm
- net /D_2_N: track 0.00 -> 51.1 mm
- net /2108_Block A/RI232_3: track 0.00 -> 50.7 mm
- net /2108_Block A/RTS232_3: track 0.00 -> 46.0 mm, vias 0 -> 2
- net /2108_Block A/DTR232_3: track 0.00 -> 45.7 mm
- net /2108_Block A/RXD1: track 0.00 -> 45.1 mm
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
Commit message: brd l
Routing:
- net /2108_Block A/TXD232_3: track 111.8 -> 31.9 mm, vias 4 -> 2
- net /2108_Block A/RXD232_3: track 115.0 -> 38.1 mm
- net /2108_Block A/RXD232_2: track 0.00 -> 38.2 mm
- net /2108_Block A/DSR232_3: track 68.2 -> 34.6 mm
- net /2108_Block A/DCD232_3: track 64.7 -> 32.3 mm, vias 2 -> 1
- net /2108_Block A/CTS232_3: track 59.6 -> 29.8 mm, vias 2 -> 1
- net /2108_Block A/RI232_3: track 50.7 -> 25.3 mm
- net /2108_Block A/RTS232_3: track 46.0 -> 23.0 mm, vias 2 -> 1
- net /2108_Block A/DTR232_3: track 45.7 -> 22.9 mm
- net Net-(J5-Pad2): track 0.00 -> 12.3 mm
- net Net-(J6-Pad2): track 24.5 -> 13.3 mm
- net Net-(J5-Pad5): track 0.00 -> 7.52 mm
- net Net-(J6-Pad5): track 14.2 -> 7.52 mm
- net /2108_Block A/TXD232_2: track 0.00 -> 5.87 mm
- net Net-(C30-Pad1): track 9.43 -> 4.72 mm
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