File: KiCad/triple_cp2108/triple_cp2108.kicad_pcb (KiCad board)
At the start: 2 copper layers, 254 parts, among them IC1 CP2108-B03-GMR, IC2 CP2108-B03-GMR, IC3 CP2108-B03-GMR, J1 USB_B, J10 DB9_Male, J11 DB9_Male, J12 RJ25, J13 RJ25, J14 RJ25, J15 RJ25, J16 DB9_Male, J17 DB9_Male, J18 DB9_Male, J19 DB9_Male, J2 USB_A, J20 RJ25, J21 RJ25, J22 RJ25, J23 RJ25, J24 DB9_Male, J25 DB9_Male, J26 DB9_Male, J27 DB9_Male, J3 Conn_02x20_Odd_Even, J4 RJ25, J5 RJ25, J6 RJ25, J7 RJ25, J8 DB9_Male, J9 DB9_Male, U1 MIC5504-3.3YM5, U10 SP3243, U11 SP3243, U12 SP3243, U13 SP3243, U14 SP3243, U2 USB2514B_Bi, U3 SP3243, U4 SP3243, U5 SP3243, U6 SP3243, U7 SP3243, U8 SP3243, U9 SP3243, Y1 24M

Commit message: 2
Routing:
- net /2108_Block A/TXD232_2: track 5.87 -> 54.9 mm, vias 0 -> 2
- net /2108_Block A/DSR232_2: track 0.00 -> 34.3 mm
- net /2108_Block A/DCD232_2: track 0.00 -> 32.4 mm, vias 0 -> 1
- net /2108_Block A/CTS232_2: track 0.00 -> 29.7 mm, vias 0 -> 1
- net /2108_Block A/RI232_2: track 0.00 -> 24.9 mm
- net /2108_Block A/DTR232_2: track 0.00 -> 23.1 mm
- net /2108_Block A/RTS232_2: track 0.00 -> 23.0 mm, vias 0 -> 1
- net /2108_Block A/RXD232_2: track 38.2 -> 56.5 mm
- net Net-(C27-Pad1): track 6.15 -> 2.73 mm
- net /2108_Block A/RXD232_3: track 38.1 -> 40.3 mm
- net Net-(D16-Pad2): track 0.00 -> 2.21 mm
- net Net-(D15-Pad2): track 0.00 -> 2.21 mm
- net /2108_Block A/TXD232_3: track 31.9 -> 30.6 mm
- net /2108_Block A/RI232_3: track 25.3 -> 24.3 mm
- net /2108_Block A/DSR232_3: track 34.6 -> 33.8 mm

Commit message: 1
Parts:
- moved D5 95.1 mm to (109.5, 67.1), turned to 270 degrees
- moved D4 94.9 mm to (109.5, 64.5), turned to 90 degrees
- moved C11 74.8 mm to (92.2, 67.9)
- moved C16 74.8 mm to (92.2, 69.9)
- moved C10 74.8 mm to (92.2, 70.0)
- moved C15 74.8 mm to (92.2, 67.9)
Connections:
- net /D_1_N renamed /D-_1
- net /D_1_P renamed /D+_1
- net /D_2_N renamed /D-_2
- net /D_2_P renamed /D+_2
- net /D_3_N renamed /D-_3
- net /D_3_P renamed /D+_3
- net /D_4_N renamed /D-_4
- net /D_4_P renamed /D+_4
- net /D_UPSTREAM_N renamed /D-_UPSTREAM
- net /D_UPSTREAM_P renamed /D+_UPSTREAM
- IC1 pad 23: /2108_Block A/RXD3_LED -> /2108_Block A/RXD4_LED
- IC1 pad 26: /2108_Block A/TXD3_LED -> /2108_Block A/TXD4_LED
- IC2 pad 23: /2108_Block B/RXD3_LED -> /2108_Block B/RXD4_LED
- IC2 pad 26: /2108_Block B/TXD3_LED -> /2108_Block B/TXD4_LED
- IC3 pad 23: /2108_Block C/RXD3_LED -> /2108_Block C/RXD4_LED
- IC3 pad 26: /2108_Block C/TXD3_LED -> /2108_Block C/TXD4_LED
Routing:
- net /2108_Block A/RXD232_4: track 0.00 -> 57.1 mm
- net /2108_Block A/TXD232_4: track 0.00 -> 55.6 mm, vias 0 -> 2
- net /2108_Block A/TXD4: track 0.00 -> 40.2 mm, vias 0 -> 4
- net /2108_Block A/DSR232_4: track 0.00 -> 34.1 mm
- net /2108_Block A/DCD232_4: track 0.00 -> 32.2 mm, vias 0 -> 1
- net /2108_Block A/CTS232_4: track 0.00 -> 30.2 mm, vias 0 -> 1
- net /2108_Block A/DTR2: track 0.00 -> 29.9 mm, vias 0 -> 2
- net /2108_Block A/RI2: track 0.00 -> 29.9 mm, vias 0 -> 2
- net /2108_Block A/DCD2: track 0.00 -> 26.2 mm, vias 0 -> 2
- net /2108_Block A/RTS2: track 0.00 -> 25.4 mm, vias 0 -> 2
- net /2108_Block A/DSR2: track 0.00 -> 25.3 mm, vias 0 -> 2
- net /2108_Block A/RI232_4: track 0.00 -> 25.3 mm
- net /2108_Block A/TXD232_3: track 30.6 -> 54.6 mm
- net /2108_Block A/RXD4: track 7.18 -> 30.4 mm, vias 1 -> 2
- net /2108_Block A/DTR232_4: track 0.00 -> 23.0 mm
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
Commit message: 2
Parts:
- C15, C16, R6: moved to B.Cu
- moved C8 81.5 mm to (93.8, 69.3), turned to 180 degrees
- moved C9 79.3 mm to (93.8, 67.2), turned to 180 degrees
- moved R6 9.01 mm to (91.9, 70.1), turned to 180 degrees
- moved C11 8.67 mm to (100.0, 64.0), turned to 90 degrees
- moved C10 8.23 mm to (97.9, 64.0), turned to 90 degrees
- moved C16 3.92 mm to (91.9, 66.0)
- moved C36 0.80 mm to (109.7, 73.9)
- moved C15 0.35 mm to (91.9, 68.1)
Routing:
- net /2108_Block A/3V3_NET: track 28.7 -> 131.6 mm, vias 0 -> 18
- net /2108_Block A/DTR4: track 0.00 -> 55.3 mm, vias 0 -> 2
- net /2108_Block A/RTS4: track 0.00 -> 50.9 mm, vias 0 -> 2
- net /2108_Block A/RI4: track 0.00 -> 33.7 mm, vias 0 -> 2
- net /2108_Block A/DSR4: track 0.00 -> 32.5 mm, vias 0 -> 2
- net /2108_Block A/DCD4: track 0.00 -> 32.4 mm, vias 0 -> 2
- net /2108_Block A/CTS4: track 0.00 -> 31.1 mm, vias 0 -> 2
- net Net-(IC1-Pad64): track 4.25 -> 10.8 mm, vias 0 -> 1
- net /VBUS_5V: track 2.08 -> 6.77 mm
- net /2108_Block A/RXD4: track 30.4 -> 28.2 mm
- net /2108_Block A/TXD4: track 40.2 -> 40.9 mm, vias 4 -> 2

Commit message: layout revert
Parts:
- C10, C11, C19, C23: moved to F.Cu
- C17, C18, C20, C21, C22, C24, C25, C26, IC1, U3, U4: moved to B.Cu
- moved C17 20.1 mm to (37.6, 87.0), turned to 270 degrees
- moved U3 19.3 mm to (43.5, 82.0), turned to 0 degrees
- moved C22 17.7 mm to (83.0, 88.1), turned to 270 degrees
- moved C19 17.3 mm to (43.3, 84.7), turned to 270 degrees
- moved C20 16.3 mm to (41.0, 88.8), turned to 180 degrees
- moved C18 15.9 mm to (50.0, 87.4), turned to 270 degrees
- moved C25 15.2 mm to (50.0, 83.4), turned to 270 degrees
- moved C26 12.2 mm to (83.8, 83.6), turned to 270 degrees
- moved C15 10.6 mm to (102.5, 68.2)
- moved C16 10.6 mm to (102.5, 66.1)
- moved C8 10.6 mm to (104.4, 69.4)
- moved C9 10.6 mm to (104.4, 67.3)
- moved R6 10.6 mm to (102.5, 70.2)
- moved C24 7.32 mm to (72.5, 89.6), turned to 0 degrees
- moved IC1 6.27 mm to (85.9, 64.8)
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Routing:
- net /2108_Block A/DTR4: track 55.3 -> 0.00 mm, vias 2 -> 0
- net /2108_Block A/RTS4: track 50.9 -> 0.00 mm, vias 2 -> 0
- net /2108_Block A/3V3_NET: track 131.6 -> 81.7 mm, vias 18 -> 4
- net /2108_Block A/TXD232_2: track 54.9 -> 5.87 mm, vias 2 -> 0
- net /2108_Block A/RXD1: track 45.1 -> 0.00 mm
- net /2108_Block A/TXD1: track 43.8 -> 0.00 mm
- net /2108_Block A/CTS1: track 42.2 -> 0.00 mm
- net /2108_Block A/TXD4: track 40.9 -> 0.00 mm, vias 2 -> 0
- net /2108_Block A/RTS1: track 40.5 -> 0.00 mm, vias 2 -> 0
- net /2108_Block A/DTR1: track 39.4 -> 0.00 mm, vias 2 -> 0
- net /2108_Block A/DSR1: track 35.4 -> 0.00 mm
- net /2108_Block A/DSR232_1: track 34.6 -> 0.00 mm
- net /2108_Block A/DSR232_2: track 34.3 -> 0.00 mm
- net /2108_Block A/RI4: track 33.7 -> 0.00 mm, vias 2 -> 0
- net /2108_Block A/DCD1: track 33.2 -> 0.00 mm
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
Commit message: 3
Parts:
- C23: moved to B.Cu
- moved C23 8.21 mm to (85.1, 85.8)
- moved U4 2.70 mm to (77.1, 79.9)
- moved C26 2.64 mm to (84.9, 81.2)
- moved C24 2.41 mm to (72.3, 87.2)
- moved C21 2.19 mm to (71.0, 84.2)
- moved C22 1.30 mm to (83.0, 86.8)
Routing:
- net /2108_Block A/RXD232_2: track 33.4 -> 5.87 mm, vias 1 -> 0
- net Net-(C24-Pad1): track 4.93 -> 0.00 mm
- net Net-(C23-Pad2): track 3.92 -> 0.00 mm, vias 1 -> 0
- net Net-(C23-Pad1): track 3.90 -> 0.00 mm, vias 1 -> 0
- net Net-(C21-Pad1): track 3.55 -> 0.00 mm
- net Net-(C24-Pad2): track 2.79 -> 0.00 mm
- net Net-(C22-Pad1): track 2.67 -> 0.00 mm

Commit message: 3
Parts:
- C19, C27, C28, C30, U5: moved to B.Cu
- C25, C26: moved to F.Cu
- moved C19 23.8 mm to (67.1, 83.3)
- moved C17 18.1 mm to (55.2, 82.8)
- moved U3 17.7 mm to (61.1, 79.9)
- moved C20 15.4 mm to (56.3, 87.2)
- moved C28 15.1 mm to (96.5, 86.6), turned to 0 degrees
- moved C18 14.5 mm to (64.5, 86.6), turned to 0 degrees
- moved C25 13.2 mm to (62.2, 78.5)
- moved C29 7.80 mm to (99.1, 83.3), turned to 270 degrees
- moved C26 7.20 mm to (78.2, 78.5)
- moved C35 5.31 mm to (94.2, 78.5), turned to 270 degrees
- moved C30 4.92 mm to (88.3, 87.2), turned to 180 degrees
- moved C27 3.80 mm to (87.2, 82.8), turned to 270 degrees
- moved C23 3.22 mm to (83.1, 83.3)
- moved C22 2.49 mm to (80.5, 86.6), turned to 0 degrees
- moved U5 1.60 mm to (93.1, 79.9), turned to 0 degrees
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Routing:
- net /2108_Block A/RXD232_3: track 56.6 -> 5.87 mm
- net /2108_Block A/TXD232_3: track 54.6 -> 5.87 mm, vias 2 -> 0
- net /2108_Block A/RXD1: track 0.00 -> 45.2 mm, vias 0 -> 2
- net /2108_Block A/CTS1: track 0.00 -> 43.5 mm, vias 0 -> 2
- net /2108_Block A/DTR1: track 0.00 -> 40.8 mm
- net /2108_Block A/TXD1: track 0.00 -> 40.5 mm
- net /2108_Block A/DSR1: track 0.00 -> 40.4 mm
- net /2108_Block A/RTS1: track 0.00 -> 40.3 mm, vias 0 -> 2
- net /2108_Block A/DCD1: track 0.00 -> 37.9 mm
- net /2108_Block A/DCD232_2: track 0.00 -> 37.0 mm
- net /2108_Block A/DCD232_1: track 0.00 -> 36.6 mm
- net /2108_Block A/DSR232_2: track 0.00 -> 34.3 mm
- net /2108_Block A/TXD232_2: track 5.87 -> 40.1 mm, vias 0 -> 1
- net /2108_Block A/DSR232_1: track 0.00 -> 34.1 mm
- net /2108_Block A/DSR232_3: track 33.8 -> 0.00 mm
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- added copper zone on B.Cu, net /2108_Block A/3V3_NET
- added copper zone on F.Cu, net /2108_Block A/3V3_NET

Commit message: 4
Parts:
- C31, C32, C34, U6: moved to B.Cu
- moved C8 16.0 mm to (104.2, 53.4)
- moved C15 16.0 mm to (102.3, 52.2)
- moved C16 16.0 mm to (102.3, 50.1)
- moved C9 16.0 mm to (104.2, 51.3)
- moved R6 16.0 mm to (102.3, 54.2)
- moved C32 15.1 mm to (112.5, 86.6), turned to 0 degrees
- moved D4 8.74 mm to (110.3, 55.8)
- moved D5 8.74 mm to (110.3, 58.4)
- moved C33 7.80 mm to (115.1, 83.3), turned to 270 degrees
- moved C10 6.53 mm to (92.4, 63.6), turned to 90 degrees
- moved C11 5.16 mm to (94.5, 63.6), turned to 90 degrees
- moved C34 4.92 mm to (104.3, 87.2), turned to 180 degrees
- moved C36 4.60 mm to (110.2, 78.5), turned to 270 degrees
- moved C31 3.80 mm to (103.2, 82.8), turned to 270 degrees
- moved U6 1.60 mm to (109.1, 79.9), turned to 0 degrees
Routing:
- net /2108_Block A/DCD232_3: track 0.00 -> 35.9 mm
- net /2108_Block A/DSR232_3: track 0.00 -> 34.0 mm
- net /2108_Block A/RTS232_3: track 0.00 -> 33.9 mm
- net /2108_Block A/TXD232_3: track 5.87 -> 38.6 mm, vias 0 -> 1
- net /2108_Block A/DTR232_3: track 0.00 -> 31.6 mm, vias 0 -> 1
- net /2108_Block A/CTS4: track 0.00 -> 31.5 mm, vias 0 -> 2
- net /2108_Block A/RXD232_3: track 5.87 -> 35.5 mm
- net /2108_Block A/DSR4: track 0.00 -> 28.5 mm
- net /2108_Block A/DCD4: track 0.00 -> 28.2 mm
- net /2108_Block A/RI4: track 0.00 -> 27.9 mm
- net /2108_Block A/RI232_3: track 0.00 -> 26.8 mm, vias 0 -> 1
- net /2108_Block A/RXD4: track 16.2 -> 42.5 mm, vias 2 -> 0
- net /2108_Block A/CTS232_3: track 0.00 -> 26.1 mm
- net /2108_Block A/TXD4: track 0.00 -> 22.7 mm, vias 0 -> 2
- net /2108_Block A/RXD232_4: track 57.1 -> 35.5 mm
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
Commit message: 5
Parts:
- C46, C47, C49, U7: moved to B.Cu
- moved C42 170.5 mm to (79.0, 62.7), turned to 0 degrees
- moved C47 15.1 mm to (128.5, 86.6), turned to 0 degrees
- moved C48 7.80 mm to (131.1, 83.3), turned to 270 degrees
- moved C54 5.31 mm to (126.2, 78.5), turned to 270 degrees
- moved C49 4.92 mm to (120.3, 87.2), turned to 180 degrees
- moved C46 3.80 mm to (119.2, 82.8), turned to 270 degrees
- moved U7 1.60 mm to (125.1, 79.9), turned to 0 degrees
- moved C10 0.51 mm to (92.4, 64.1)
- moved C11 0.51 mm to (94.5, 64.1)
Routing:
- net /2108_Block A/3V3_NET: track 75.3 -> 141.6 mm, vias 9 -> 15
- net /2108_Block A/RXD232_4: track 35.5 -> 58.0 mm
- net /2108_Block A/RXD232_1: track 36.8 -> 59.3 mm
- net /2108_Block A/RXD232_3: track 35.5 -> 57.8 mm
- net /2108_Block A/RXD232_2: track 36.8 -> 58.9 mm
- net /2108_Block A/TXD232_1: track 39.0 -> 60.5 mm
- net /2108_Block A/TXD232_2: track 40.1 -> 61.0 mm
- net /2108_Block A/TXD232_4: track 38.8 -> 59.5 mm
- net /2108_Block A/TXD232_3: track 38.6 -> 59.1 mm
- net /2108_Block A/RXD2: track 25.9 -> 31.3 mm
