File: KiCad/triple_cp2108/triple_cp2108.kicad_pcb (KiCad board)
At the start: 2 copper layers, 254 parts, among them IC1 CP2108-B03-GMR, IC2 CP2108-B03-GMR, IC3 CP2108-B03-GMR, J1 USB_B, J10 DB9_Male, J11 DB9_Male, J12 RJ25, J13 RJ25, J14 RJ25, J15 RJ25, J16 DB9_Male, J17 DB9_Male, J18 DB9_Male, J19 DB9_Male, J2 USB_A, J20 RJ25, J21 RJ25, J22 RJ25, J23 RJ25, J24 DB9_Male, J25 DB9_Male, J26 DB9_Male, J27 DB9_Male, J3 Conn_02x20_Odd_Even, J4 RJ25, J5 RJ25, J6 RJ25, J7 RJ25, J8 DB9_Male, J9 DB9_Male, U1 MIC5504-3.3YM5, U10 SP3243, U11 SP3243, U12 SP3243, U13 SP3243, U14 SP3243, U2 USB2514B_Bi, U3 SP3243, U4 SP3243, U5 SP3243, U6 SP3243, U7 SP3243, U8 SP3243, U9 SP3243, Y1 24M

Commit message: 5
Parts:
- C50, C51, C53, C56, C57, C59, C60, C61, C63, C75, C76, C78, C79, C80, C82, C85, C86, C88, C89, C90, C92, IC2, IC3, U10, U11, U12, U13, U14, U8, U9: moved to B.Cu
- moved U2 46.9 mm to (77.0, 36.7)
- moved C51 15.1 mm to (144.5, 86.6), turned to 0 degrees
- moved C57 15.1 mm to (160.5, 86.6), turned to 0 degrees
- moved C61 15.1 mm to (176.5, 86.6), turned to 0 degrees
- moved C76 15.1 mm to (192.5, 86.6), turned to 0 degrees
- moved C80 15.1 mm to (208.5, 86.6), turned to 0 degrees
- moved C86 15.1 mm to (224.5, 86.6), turned to 0 degrees
- moved C90 15.1 mm to (240.5, 86.6), turned to 0 degrees
- moved C52 7.80 mm to (147.1, 83.3), turned to 270 degrees
- moved C58 7.80 mm to (163.1, 83.3), turned to 270 degrees
- moved C62 7.80 mm to (179.1, 83.3), turned to 270 degrees
- moved C77 7.80 mm to (195.1, 83.3), turned to 270 degrees
- moved C81 7.80 mm to (211.1, 83.3), turned to 270 degrees
- moved C87 7.80 mm to (227.1, 83.3), turned to 270 degrees
- moved C91 7.80 mm to (243.1, 83.3), turned to 270 degrees
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Routing:
- net /D+_3: track 115.8 -> 0.00 mm
- net /D-_3: track 115.8 -> 0.00 mm
- net /2108_Block B/3V3_NET: track 0.00 -> 56.6 mm
- net /D+_2: track 51.1 -> 0.00 mm
- net /D-_2: track 51.1 -> 0.00 mm
- net /D-_4: track 20.0 -> 0.00 mm
- net /D+_4: track 18.3 -> 0.00 mm

Commit message: 6
Routing:
- net /2108_Block B/TXD232_1: track 0.00 -> 59.8 mm, vias 0 -> 1
- net /2108_Block B/RXD232_1: track 0.00 -> 59.0 mm
- net /2108_Block C/3V3_NET: track 0.00 -> 56.5 mm
- net /2108_Block B/DCD232_1: track 0.00 -> 35.2 mm
- net /2108_Block B/DSR232_1: track 0.00 -> 34.4 mm
- net /2108_Block B/RTS232_1: track 0.00 -> 33.4 mm
- net /2108_Block B/DTR232_1: track 0.00 -> 31.9 mm, vias 0 -> 1
- net /2108_Block C/RXD232_3: track 0.00 -> 28.5 mm
- net /2108_Block C/RXD232_2: track 0.00 -> 28.5 mm
- net /2108_Block B/RXD232_2: track 0.00 -> 28.4 mm
- net /2108_Block C/RXD232_4: track 0.00 -> 28.4 mm
- net /2108_Block C/RXD232_1: track 0.00 -> 28.4 mm
- net /2108_Block B/RXD232_4: track 0.00 -> 28.4 mm
- net /2108_Block B/RXD232_3: track 0.00 -> 28.4 mm
- net /2108_Block B/RI232_1: track 0.00 -> 26.9 mm, vias 0 -> 1
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
Commit message: 7
Parts:
- moved C42 62.0 mm to (141.0, 61.2)
- moved C12 34.6 mm to (54.4, 53.1)
- moved C13 19.4 mm to (48.0, 56.8)
- moved C14 16.8 mm to (53.8, 57.1)
Routing:
- net /2108_Block C/TXD232_1: track 5.87 -> 60.1 mm, vias 0 -> 1
- net /2108_Block B/TXD232_4: track 5.87 -> 60.1 mm, vias 0 -> 1
- net /2108_Block B/TXD232_2: track 5.87 -> 60.0 mm, vias 0 -> 1
- net /2108_Block B/TXD232_3: track 5.87 -> 59.9 mm, vias 0 -> 1
- net /2108_Block C/TXD232_2: track 5.87 -> 59.6 mm, vias 0 -> 1
- net /2108_Block C/TXD232_3: track 5.87 -> 59.0 mm, vias 0 -> 1
- net /2108_Block C/TXD232_4: track 5.87 -> 58.4 mm, vias 0 -> 1
- net /2108_Block B/DCD232_2: track 0.00 -> 35.2 mm
- net /2108_Block B/DCD232_3: track 0.00 -> 35.0 mm
- net /2108_Block C/DCD232_3: track 0.00 -> 34.6 mm
- net /2108_Block C/DCD232_1: track 0.00 -> 34.6 mm
- net /2108_Block C/DCD232_4: track 0.00 -> 34.6 mm
- net /2108_Block C/DCD232_2: track 0.00 -> 34.6 mm
- net /2108_Block B/DCD232_4: track 0.00 -> 34.6 mm
- net /2108_Block B/DSR232_2: track 0.00 -> 33.9 mm
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
Commit message: 9
Parts:
- moved C13 41.3 mm to (86.1, 72.6)
- moved C14 39.4 mm to (92.7, 63.8), turned to 90 degrees
- moved C12 27.1 mm to (79.5, 63.2), turned to 270 degrees
- moved C11 12.9 mm to (83.6, 57.3), turned to 270 degrees
- moved C10 9.58 mm to (85.7, 57.3), turned to 270 degrees
- moved C19 7.69 mm to (68.1, 75.7), turned to 45 degrees
Routing:
- net /2108_Block A/TXD1_LED: track 2.73 -> 75.1 mm, vias 1 -> 3
- net /2108_Block A/RXD1_LED: track 4.68 -> 73.5 mm, vias 0 -> 3
- net /2108_Block A/TXD2_LED: track 0.00 -> 64.1 mm, vias 0 -> 1
- net /2108_Block A/RXD2_LED: track 0.00 -> 61.9 mm, vias 0 -> 1
- net /2108_Block A/~SUSPEND: track 0.00 -> 60.1 mm, vias 0 -> 4
- net Net-(C19-Pad2): track 2.45 -> 11.5 mm
- net /2108_Block A/3V3_NET: track 143.4 -> 138.9 mm, vias 16 -> 13
- net Net-(C19-Pad1): track 2.67 -> 6.99 mm
- net /IO4: track 0.00 -> 3.14 mm
- net /2108_Block A/RXD2: track 31.3 -> 28.6 mm, vias 2 -> 4
- net /IO3: track 0.00 -> 2.38 mm
- net GND: vias 0 -> 48
- added copper zone on F.Cu, net GND

Commit message: 9
Parts:
- C8, C9, D4, D5: moved to B.Cu
- moved U2 29.8 mm to (106.7, 33.8)
- moved C15 21.8 mm to (80.6, 53.4)
- moved C16 21.8 mm to (80.6, 51.4)
- moved D5 19.2 mm to (91.2, 56.0), turned to 90 degrees
- moved D4 19.2 mm to (91.2, 57.8), turned to 270 degrees
- moved C8 18.7 mm to (85.9, 56.6), turned to 315 degrees
- moved C9 16.6 mm to (88.3, 56.0), turned to 315 degrees
- moved R6 10.7 mm to (93.2, 59.8), turned to 0 degrees
- moved C11 4.31 mm to (86.9, 60.0), turned to 90 degrees
- moved C12 3.10 mm to (81.3, 65.8), turned to 180 degrees
- moved C13 3.08 mm to (85.9, 69.6), turned to 270 degrees
- moved C14 2.94 mm to (90.3, 62.1), turned to 0 degrees
- moved C10 2.88 mm to (84.8, 60.0), turned to 90 degrees
Routing:
- net /2108_Block A/3V3_NET: track 138.9 -> 245.9 mm, vias 13 -> 17
- net /2108_Block A/TXD4_LED: track 0.00 -> 94.0 mm, vias 0 -> 3
- net /2108_Block A/RXD4_LED: track 0.00 -> 92.8 mm, vias 0 -> 3
- net /2108_Block A/TXD3_LED: track 0.00 -> 77.3 mm, vias 0 -> 3
- net /2108_Block A/RXD3_LED: track 0.00 -> 75.5 mm, vias 0 -> 3
- net /2108_Block B/RXD1_LED: track 0.00 -> 50.6 mm, vias 0 -> 1
- net /2108_Block B/TXD1_LED: track 0.00 -> 48.3 mm, vias 0 -> 1
- net /IO8: track 0.00 -> 24.7 mm, vias 0 -> 2
- net /IO7: track 0.00 -> 21.5 mm, vias 0 -> 2
- net /IO6: track 0.00 -> 16.3 mm, vias 0 -> 2
- net /IO5: track 0.00 -> 14.3 mm, vias 0 -> 2
- net /2108_Block A/~SUSPEND: track 60.1 -> 72.0 mm, vias 4 -> 5
- net /IO2: track 1.46 -> 9.72 mm, vias 0 -> 2
- net /2108_Block B/TXD2_LED: track 0.00 -> 8.25 mm, vias 0 -> 1
- net /VBUS_5V: track 2.08 -> 10.1 mm
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
Commit message: 10
Parts:
- moved C42 15.1 mm to (127.6, 54.2)
Routing:
- net /2108_Block B/RXD4_LED: track 0.00 -> 51.8 mm, vias 0 -> 1
- net /2108_Block B/TXD4_LED: track 0.00 -> 51.5 mm, vias 0 -> 1
- net /2108_Block B/TXD3_LED: track 0.00 -> 51.1 mm, vias 0 -> 1
- net /2108_Block B/RXD3_LED: track 0.00 -> 48.5 mm, vias 0 -> 1
- net /2108_Block B/TXD2_LED: track 8.25 -> 54.2 mm
- net /2108_Block B/RXD2_LED: track 6.75 -> 49.6 mm
- net /2108_Block B/TXD1: track 0.00 -> 40.9 mm
- net /2108_Block B/RTS1: track 0.00 -> 39.9 mm
- net /2108_Block B/RXD1: track 0.00 -> 39.5 mm, vias 0 -> 2
- net /2108_Block B/CTS1: track 0.00 -> 38.2 mm, vias 0 -> 2
- net /2108_Block B/DTR1: track 0.00 -> 37.3 mm
- net /2108_Block B/RXD4: track 0.00 -> 34.6 mm
- net /2108_Block B/DSR1: track 0.00 -> 33.8 mm
- net /2108_Block B/CTS4: track 0.00 -> 33.3 mm
- net /2108_Block B/DCD1: track 0.00 -> 31.5 mm
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
Commit message: in prgs.
Routing:
- net /2108_Block B/~SUSPEND: track 0.00 -> 71.2 mm, vias 0 -> 5
- net /2108_Block B/3V3_NET: track 58.4 -> 119.7 mm, vias 1 -> 9
- net /2108_Block B/TXD4_LED: track 51.5 -> 88.2 mm, vias 1 -> 3
- net /2108_Block B/RXD4_LED: track 51.8 -> 86.5 mm, vias 1 -> 3
- net /2108_Block B/RXD3_LED: track 48.5 -> 75.0 mm, vias 1 -> 3
- net /2108_Block B/TXD3_LED: track 51.1 -> 75.8 mm, vias 1 -> 3
- net /2108_Block B/RXD2_LED: track 49.6 -> 62.0 mm
- net /2108_Block B/TXD2_LED: track 54.2 -> 64.2 mm
- net /IO13: track 0.00 -> 3.94 mm, vias 0 -> 1
- net /IO12: track 0.00 -> 3.36 mm, vias 0 -> 1
- net /IO10: track 4.77 -> 1.45 mm, vias 0 -> 1
- net /IO9: track 4.39 -> 1.63 mm, vias 0 -> 1
- net /IO14: track 0.00 -> 2.75 mm, vias 0 -> 1
- net /IO15: track 0.00 -> 2.28 mm, vias 0 -> 1
- net /IO11: track 0.00 -> 1.76 mm, vias 0 -> 1
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- added copper zone on B.Cu, net /2108_Block B/3V3_NET
- added copper zone on F.Cu, net /2108_Block B/3V3_NET
